File: segment_TEST/segment_TEST.sch (KiCad schematic (older format))
At the start: 80 parts, among them J1 COL0, J10 COL9, J11 COL10, J12 COL11, J13 COL12, J14 COL13, J15 ROWS, J2 COL1, J3 COL2, J4 COL3, J5 COL4, J6 COL5, J7 COL6, J8 COL7, J9 COL8, SW1 SW_Push_45deg, SW10 SW_Push_45deg, SW11 SW_Push_45deg, SW12 SW_Push_45deg, SW13 SW_Push_45deg, SW14 SW_Push_45deg, SW15 SW_Push_45deg, SW16 SW_Push_45deg, SW17 SW_Push_45deg, SW18 SW_Push_45deg, SW19 SW_Push_45deg, SW2 SW_Push_45deg, SW20 SW_Push_45deg, SW21 SW_Push_45deg, SW22 SW_Push_45deg, SW23 SW_Push_45deg, SW24 SW_Push_45deg, SW25 SW_Push_45deg, SW26 SW_Push_45deg, SW27 SW_Push_45deg, SW28 SW_Push_45deg, SW29 SW_Push_45deg, SW3 SW_Push_45deg, SW30 SW_Push_45deg, SW31 SW_Push_45deg, SW32 SW_Push_45deg, SW33 SW_Push_45deg, SW34 SW_Push_45deg, SW35 SW_Push_45deg, SW36 SW_Push_45deg, SW37 SW_Push_45deg, SW38 SW_Push_45deg, SW39 SW_Push_45deg, SW4 SW_Push_45deg, SW40 SW_Push_45deg, SW41 SW_Push_45deg, SW42 SW_Push_45deg, SW43 SW_Push_45deg, SW44 SW_Push_45deg, SW45 SW_Push_45deg, SW46 SW_Push_45deg, SW47 SW_Push_45deg, SW48 SW_Push_45deg, SW49 SW_Push_45deg, SW5 SW_Push_45deg, SW50 SW_Push_45deg, SW51 SW_Push_45deg, SW52 SW_Push_45deg, SW53 SW_Push_45deg, SW54 SW_Push_45deg, SW55 SW_Push_45deg, SW56 SW_Push_45deg, SW57 SW_Push_45deg, SW58 SW_Push_45deg, SW59 SW_Push_45deg, SW6 SW_Push_45deg, SW60 SW_Push_45deg, SW61 SW_Push_45deg, SW62 SW_Push_45deg, SW63 SW_Push_45deg, SW64 SW_Push_45deg, SW65 SW_Push_45deg, SW7 SW_Push_45deg, SW8 SW_Push_45deg, SW9 SW_Push_45deg

Commit message: Completed test board layout; implementing option footprints
Parts:
- SW1, SW10, SW11, SW12, SW13, SW16, SW17, SW18, SW19, SW2, SW20, SW21, SW22, SW23, SW24, SW25, SW26, SW27, SW28, SW3, SW30, SW31, SW32, SW33, SW34, SW35, SW36, SW37, SW38, SW39, SW4, SW40, SW44, SW45, SW46, SW47, SW48, SW49, SW5, SW50, SW51, SW52, SW53, SW54, SW56, SW58, SW6, SW64, SW7, SW8, SW9: footprint Button_Switch_Keyboard:SW_Cherry_MX_1.00u_PCB -> Segment_Footprints:Segment_MX_1.00u_PCB
- SW14: footprint Button_Switch_Keyboard:SW_Cherry_MX_1.00u_PCB -> Segment_Footprints:Segment_MX_1.00u_2.00u_PCB
- SW15, SW42, SW57, SW59, SW63, SW65: footprint Button_Switch_Keyboard:SW_Cherry_MX_1.50u_PCB -> Segment_Footprints:Segment_MX_1.50u_PCB
- SW29, SW55: footprint Button_Switch_Keyboard:SW_Cherry_MX_1.75u_PCB -> Segment_Footprints:Segment_MX_1.75u_PCB
- SW41: footprint Button_Switch_Keyboard:SW_Cherry_MX_2.25u_PCB -> Segment_Footprints:Segment_MX_2.25u_PCB
- SW43: footprint Button_Switch_Keyboard:SW_Cherry_MX_1.25u_PCB -> Segment_Footprints:Segment_MX_1.25u_2.25u_PCB
- SW60, SW62: footprint Button_Switch_Keyboard:SW_Cherry_MX_2.75u_PCB -> Segment_Footprints:Segment_MX_2.75u_PCB
- SW61: footprint Button_Switch_Keyboard:SW_Cherry_MX_1.50u_PCB -> Segment_Footprints:Segment_MX_7.00u_PCB

Commit message: Layout mostly complete for test board
Parts:
- J1, J10, J12, J13, J14, J15, J2, J3, J6, J8: footprint Connector_PinHeader_2.54mm:PinHeader_1x05_P2.54mm_Vertical -> Connector_PinHeader_2.54mm:PinHeader_1x06_P2.54mm_Vertical
- J11, J4, J5, J7, J9: footprint Connector_PinHeader_2.54mm:PinHeader_1x04_P2.54mm_Vertical -> Connector_PinHeader_2.54mm:PinHeader_1x06_P2.54mm_Vertical
- SW29: footprint Segment_Footprints:Segment_MX_1.75u_PCB -> Segment_Footprints:Segment_MX_1.25u_1.75u_PCB
- SW41: footprint Segment_Footprints:Segment_MX_2.25u_PCB -> Segment_Footprints:Segment_MX_1.00u_2.25u_PCB
- SW42: footprint Segment_Footprints:Segment_MX_1.50u_PCB -> Segment_Footprints:Segment_MX_1.50u_ISO_PCB
- SW55: footprint Segment_Footprints:Segment_MX_1.75u_PCB -> Segment_Footprints:Segment_MX_1.00u_2.75u_PCB
- SW56: footprint Segment_Footprints:Segment_MX_1.00u_PCB -> Segment_Footprints:Segment_MX_1.75u_PCB
Changed lines of the file:
@@
 F 0 "J1" H 1168 1025 50  0000 C CNN
 F 1 "COL0" H 1168 1116 50  0000 C CNN
-F 2 "Connector_PinHeader_2.54mm:PinHeader_1x05_P2.54mm_Vertical" H 1250 1450 50  0001 C CNN
+F 2 "Connector_PinHeader_2.54mm:PinHeader_1x06_P2.54mm_Vertical" H 1250 1450 50  0001 C CNN
 F 3 "~" H 1250 1450 50  0001 C CNN
 	1    1250 1450
@@
 F 0 "J2" H 3168 1025 50  0000 C CNN
 F 1 "COL1" H 3168 1116 50  0000 C CNN
-F 2 "Connector_PinHeader_2.54mm:PinHeader_1x05_P2.54mm_Vertical" H 3250 1450 50  0001 C CNN
+F 2 "Connector_PinHeader_2.54mm:PinHeader_1x06_P2.54mm_Vertical" H 3250 1450 50  0001 C CNN
 F 3 "~" H 3250 1450 50  0001 C CNN
 	1    3250 1450
@@
 F 0 "J3" H 5168 1025 50  0000 C CNN
 F 1 "COL2" H 5168 1116 50  0000 C CNN
-F 2 "Connector_PinHeader_2.54mm:PinHeader_1x05_P2.54mm_Vertical" H 5250 1450 50  0001 C CNN
+F 2 "Connector_PinHeader_2.54mm:PinHeader_1x06_P2.54mm_Vertical" H 5250 1450 50  0001 C CNN
 F 3 "~" H 5250 1450 50  0001 C CNN
 	1    5250 1450
@@
 F 0 "J4" H 7168 1025 50  0000 C CNN
 F 1 "COL3" H 7168 1116 50  0000 C CNN
-F 2 "Connector_PinHeader_2.54mm:PinHeader_1x04_P2.54mm_Vertical" H 7250 1450 50  0001 C CNN
+F 2 "Connector_PinHeader_2.54mm:PinHeader_1x06_P2.54mm_Vertical" H 7250 1450 50  0001 C CNN
 F 3 "~" H 7250 1450 50  0001 C CNN
 	1    7250 1450
@@
 F 0 "J5" H 9168 1025 50  0000 C CNN
 F 1 "COL4" H 9168 1116 50  0000 C CNN
-F 2 "Connector_PinHeader_2.54mm:PinHeader_1x04_P2.54mm_Vertical" H 9250 1450 50  0001 C CNN
+F 2 "Connector_PinHeader_2.54mm:PinHeader_1x06_P2.54mm_Vertical" H 9250 1450 50  0001 C CNN
 F 3 "~" H 9250 1450 50  0001 C CNN
 	1    9250 1450
@@
 F 0 "J14" H 7168 4425 50  0000 C CNN
 F 1 "COL13" H 7168 4516 50  0000 C CNN
-F 2 "Connector_PinHeader_2.54mm:PinHeader_1x05_P2.54mm_Vertical" H 7250 4850 50  0001 C CNN
+F 2 "Connector_PinHeader_2.54mm:PinHeader_1x06_P2.54mm_Vertical" H 7250 4850 50  0001 C CNN
 F 3 "~" H 7250 4850 50  0001 C CNN
 	1    7250 4850
@@
 F 0 "SW42" V 8000 4850 50  0000 R CNN
 F 1 "SW_Push_45deg" H 7950 5140 50  0001 C CNN
-F 2 "Segment_Footprints:Segment_MX_1.50u_PCB" H 7950 4950 50  0001 C CNN
+F 2 "Segment_Footprints:Segment_MX_1.50u_ISO_PCB" H 7950 4950 50  0001 C CNN
 F 3 "~" H 7950 4950 50  0001 C CNN
 	1    7950 4950
@@
 F 0 "SW56" V 7800 4950 50  0000 R CNN
 F 1 "SW_Push_45deg" H 7750 5240 50  0001 C CNN
-F 2 "Segment_Footprints:Segment_MX_1.00u_PCB" H 7750 5050 50  0001 C CNN
+F 2 "Segment_Footprints:Segment_MX_1.75u_PCB" H 7750 5050 50  0001 C CNN
 F 3 "~" H 7750 5050 50  0001 C CNN
 	1    7750 5050
@@
 F 0 "J13" H 5168 4425 50  0000 C CNN
 F 1 "COL12" H 5168 4516 50  0000 C CNN
-F 2 "Connector_PinHeader_2.54mm:PinHeader_1x05_P2.54mm_Vertical" H 5250 4850 50  0001 C CNN
+F 2 "Connector_PinHeader_2.54mm:PinHeader_1x06_P2.54mm_Vertical" H 5250 4850 50  0001 C CNN
 F 3 "~" H 5250 4850 50  0001 C CNN
 	1    5250 4850
@@
 F 0 "SW41" V 6000 4850 50  0000 R CNN
 F 1 "SW_Push_45deg" H 5950 5140 50  0001 C CNN
-F 2 "Segment_Footprints:Segment_MX_2.25u_PCB" H 5950 4950 50  0001 C CNN
+F 2 "Segment_Footprints:Segment_MX_1.00u_2.25u_PCB" H 5950 4950 50  0001 C CNN
 F 3 "~" H 5950 4950 50  0001 C CNN
 	1    5950 4950
@@
 F 0 "SW55" V 5800 4950 50  0000 R CNN
 F 1 "SW_Push_45deg" H 5750 5240 50  0001 C CNN
-F 2 "Segment_Footprints:Segment_MX_1.75u_PCB" H 5750 5050 50  0001 C CNN
+F 2 "Segment_Footprints:Segment_MX_1.00u_2.75u_PCB" H 5750 5050 50  0001 C CNN
 F 3 "~" H 5750 5050 50  0001 C CNN
 	1    5750 5050
@@
 F 0 "J12" H 3168 4425 50  0000 C CNN
 F 1 "COL11" H 3168 4516 50  0000 C CNN
-F 2 "Connector_PinHeader_2.54mm:PinHeader_1x05_P2.54mm_Vertical" H 3250 4850 50  0001 C CNN
+F 2 "Connector_PinHeader_2.54mm:PinHeader_1x06_P2.54mm_Vertical" H 3250 4850 50  0001 C CNN
 F 3 "~" H 3250 4850 50  0001 C CNN
 	1    3250 4850
@@
 F 0 "J11" H 1168 4425 50  0000 C CNN
 F 1 "COL10" H 1168 4516 50  0000 C CNN
-F 2 "Connector_PinHeader_2.54mm:PinHeader_1x04_P2.54mm_Vertical" H 1250 4850 50  0001 C CNN
+F 2 "Connector_PinHeader_2.54mm:PinHeader_1x06_P2.54mm_Vertical" H 1250 4850 50  0001 C CNN
 F 3 "~" H 1250 4850 50  0001 C CNN
 	1    1250 4850
@@
 F 0 "J10" H 9168 2725 50  0000 C CNN
 F 1 "COL9" H 9168 2816 50  0000 C CNN
-F 2 "Connector_PinHeader_2.54mm:PinHeader_1x05_P2.54mm_Vertical" H 9250 3150 50  0001 C CNN
+F 2 "Connector_PinHeader_2.54mm:PinHeader_1x06_P2.54mm_Vertical" H 9250 3150 50  0001 C CNN
 F 3 "~" H 9250 3150 50  0001 C CNN
 	1    9250 3150
@@
 F 0 "J9" H 7168 2725 50  0000 C CNN
 F 1 "COL8" H 7168 2816 50  0000 C CNN
-F 2 "Connector_PinHeader_2.54mm:PinHeader_1x04_P2.54mm_Vertical" H 7250 3150 50  0001 C CNN
+F 2 "Connector_PinHeader_2.54mm:PinHeader_1x06_P2.54mm_Vertical" H 7250 3150 50  0001 C CNN
 F 3 "~" H 7250 3150 50  0001 C CNN
 	1    7250 3150
@@
 F 0 "J8" H 5168 2725 50  0000 C CNN
 F 1 "COL7" H 5168 2816 50  0000 C CNN
-F 2 "Connector_PinHeader_2.54mm:PinHeader_1x05_P2.54mm_Vertical" H 5250 3150 50  0001 C CNN
+F 2 "Connector_PinHeader_2.54mm:PinHeader_1x06_P2.54mm_Vertical" H 5250 3150 50  0001 C CNN
 F 3 "~" H 5250 3150 50  0001 C CNN
 	1    5250 3150
@@
 F 0 "J7" H 3168 2725 50  0000 C CNN
 F 1 "COL6" H 3168 2816 50  0000 C CNN
-F 2 "Connector_PinHeader_2.54mm:PinHeader_1x04_P2.54mm_Vertical" H 3250 3150 50  0001 C CNN
+F 2 "Connector_PinHeader_2.54mm:PinHeader_1x06_P2.54mm_Vertical" H 3250 3150 50  0001 C CNN
 F 3 "~" H 3250 3150 50  0001 C CNN
 	1    3250 3150
@@
 F 0 "J6" H 1168 2725 50  0000 C CNN
 F 1 "COL5" H 1168 2816 50  0000 C CNN
-F 2 "Connector_PinHeader_2.54mm:PinHeader_1x05_P2.54mm_Vertical" H 1250 3150 50  0001 C CNN
+F 2 "Connector_PinHeader_2.54mm:PinHeader_1x06_P2.54mm_Vertical" H 1250 3150 50  0001 C CNN
 F 3 "~" H 1250 3150 50  0001 C CNN
 	1    1250 3150
@@
 F 0 "J15" H 9168 4425 50  0000 C CNN
 F 1 "ROWS" H 9168 4516 50  0000 C CNN
-F 2 "Connector_PinHeader_2.54mm:PinHeader_1x05_P2.54mm_Vertical" H 9250 4850 50  0001 C CNN
+F 2 "Connector_PinHeader_2.54mm:PinHeader_1x06_P2.54mm_Vertical" H 9250 4850 50  0001 C CNN
 F 3 "~" H 9250 4850 50  0001 C CNN
 	1    9250 4850
@@
 F 0 "SW29" V 2000 1450 50  0000 R CNN
 F 1 "SW_Push_45deg" H 1950 1740 50  0001 C CNN
-F 2 "Segment_Footprints:Segment_MX_1.75u_PCB" H 1950 1550 50  0001 C CNN
+F 2 "Segment_Footprints:Segment_MX_1.25u_1.75u_PCB" H 1950 1550 50  0001 C CNN
 F 3 "~" H 1950 1550 50  0001 C CNN
 	1    1950 1550

Commit message: Added JST-XH connectors to test board
Parts:
- J1, J10, J11, J12, J13, J14, J15, J2, J3, J4, J5, J6, J7, J8, J9: footprint Connector_PinHeader_2.54mm:PinHeader_1x06_P2.54mm_Vertical -> Connector_JST:JST_XH_S6B-XH-A_1x06_P2.50mm_Horizontal
Changed lines of the file:
@@
 F 0 "J1" H 1168 1025 50  0000 C CNN
 F 1 "COL0" H 1168 1116 50  0000 C CNN
-F 2 "Connector_PinHeader_2.54mm:PinHeader_1x06_P2.54mm_Vertical" H 1250 1450 50  0001 C CNN
+F 2 "Connector_JST:JST_XH_S6B-XH-A_1x06_P2.50mm_Horizontal" H 1250 1450 50  0001 C CNN
 F 3 "~" H 1250 1450 50  0001 C CNN
 	1    1250 1450
@@
 F 0 "J2" H 3168 1025 50  0000 C CNN
 F 1 "COL1" H 3168 1116 50  0000 C CNN
-F 2 "Connector_PinHeader_2.54mm:PinHeader_1x06_P2.54mm_Vertical" H 3250 1450 50  0001 C CNN
+F 2 "Connector_JST:JST_XH_S6B-XH-A_1x06_P2.50mm_Horizontal" H 3250 1450 50  0001 C CNN
 F 3 "~" H 3250 1450 50  0001 C CNN
 	1    3250 1450
@@
 F 0 "J3" H 5168 1025 50  0000 C CNN
 F 1 "COL2" H 5168 1116 50  0000 C CNN
-F 2 "Connector_PinHeader_2.54mm:PinHeader_1x06_P2.54mm_Vertical" H 5250 1450 50  0001 C CNN
+F 2 "Connector_JST:JST_XH_S6B-XH-A_1x06_P2.50mm_Horizontal" H 5250 1450 50  0001 C CNN
 F 3 "~" H 5250 1450 50  0001 C CNN
 	1    5250 1450
@@
 F 0 "J4" H 7168 1025 50  0000 C CNN
 F 1 "COL3" H 7168 1116 50  0000 C CNN
-F 2 "Connector_PinHeader_2.54mm:PinHeader_1x06_P2.54mm_Vertical" H 7250 1450 50  0001 C CNN
+F 2 "Connector_JST:JST_XH_S6B-XH-A_1x06_P2.50mm_Horizontal" H 7250 1450 50  0001 C CNN
 F 3 "~" H 7250 1450 50  0001 C CNN
 	1    7250 1450
@@
 F 0 "J5" H 9168 1025 50  0000 C CNN
 F 1 "COL4" H 9168 1116 50  0000 C CNN
-F 2 "Connector_PinHeader_2.54mm:PinHeader_1x06_P2.54mm_Vertical" H 9250 1450 50  0001 C CNN
+F 2 "Connector_JST:JST_XH_S6B-XH-A_1x06_P2.50mm_Horizontal" H 9250 1450 50  0001 C CNN
 F 3 "~" H 9250 1450 50  0001 C CNN
 	1    9250 1450
@@
 F 0 "J14" H 7168 4425 50  0000 C CNN
 F 1 "COL13" H 7168 4516 50  0000 C CNN
-F 2 "Connector_PinHeader_2.54mm:PinHeader_1x06_P2.54mm_Vertical" H 7250 4850 50  0001 C CNN
+F 2 "Connector_JST:JST_XH_S6B-XH-A_1x06_P2.50mm_Horizontal" H 7250 4850 50  0001 C CNN
 F 3 "~" H 7250 4850 50  0001 C CNN
 	1    7250 4850
@@
 F 0 "J13" H 5168 4425 50  0000 C CNN
 F 1 "COL12" H 5168 4516 50  0000 C CNN
-F 2 "Connector_PinHeader_2.54mm:PinHeader_1x06_P2.54mm_Vertical" H 5250 4850 50  0001 C CNN
+F 2 "Connector_JST:JST_XH_S6B-XH-A_1x06_P2.50mm_Horizontal" H 5250 4850 50  0001 C CNN
 F 3 "~" H 5250 4850 50  0001 C CNN
 	1    5250 4850
@@
 F 0 "J12" H 3168 4425 50  0000 C CNN
 F 1 "COL11" H 3168 4516 50  0000 C CNN
-F 2 "Connector_PinHeader_2.54mm:PinHeader_1x06_P2.54mm_Vertical" H 3250 4850 50  0001 C CNN
+F 2 "Connector_JST:JST_XH_S6B-XH-A_1x06_P2.50mm_Horizontal" H 3250 4850 50  0001 C CNN
 F 3 "~" H 3250 4850 50  0001 C CNN
 	1    3250 4850
@@
 F 0 "J11" H 1168 4425 50  0000 C CNN
 F 1 "COL10" H 1168 4516 50  0000 C CNN
-F 2 "Connector_PinHeader_2.54mm:PinHeader_1x06_P2.54mm_Vertical" H 1250 4850 50  0001 C CNN
+F 2 "Connector_JST:JST_XH_S6B-XH-A_1x06_P2.50mm_Horizontal" H 1250 4850 50  0001 C CNN
 F 3 "~" H 1250 4850 50  0001 C CNN
 	1    1250 4850
@@
 F 0 "J10" H 9168 2725 50  0000 C CNN
 F 1 "COL9" H 9168 2816 50  0000 C CNN
-F 2 "Connector_PinHeader_2.54mm:PinHeader_1x06_P2.54mm_Vertical" H 9250 3150 50  0001 C CNN
+F 2 "Connector_JST:JST_XH_S6B-XH-A_1x06_P2.50mm_Horizontal" H 9250 3150 50  0001 C CNN
 F 3 "~" H 9250 3150 50  0001 C CNN
 	1    9250 3150
@@
 F 0 "J9" H 7168 2725 50  0000 C CNN
 F 1 "COL8" H 7168 2816 50  0000 C CNN
-F 2 "Connector_PinHeader_2.54mm:PinHeader_1x06_P2.54mm_Vertical" H 7250 3150 50  0001 C CNN
+F 2 "Connector_JST:JST_XH_S6B-XH-A_1x06_P2.50mm_Horizontal" H 7250 3150 50  0001 C CNN
 F 3 "~" H 7250 3150 50  0001 C CNN
 	1    7250 3150
@@
 F 0 "J8" H 5168 2725 50  0000 C CNN
 F 1 "COL7" H 5168 2816 50  0000 C CNN
-F 2 "Connector_PinHeader_2.54mm:PinHeader_1x06_P2.54mm_Vertical" H 5250 3150 50  0001 C CNN
+F 2 "Connector_JST:JST_XH_S6B-XH-A_1x06_P2.50mm_Horizontal" H 5250 3150 50  0001 C CNN
 F 3 "~" H 5250 3150 50  0001 C CNN
 	1    5250 3150
@@
 F 0 "J7" H 3168 2725 50  0000 C CNN
 F 1 "COL6" H 3168 2816 50  0000 C CNN
-F 2 "Connector_PinHeader_2.54mm:PinHeader_1x06_P2.54mm_Vertical" H 3250 3150 50  0001 C CNN
+F 2 "Connector_JST:JST_XH_S6B-XH-A_1x06_P2.50mm_Horizontal" H 3250 3150 50  0001 C CNN
 F 3 "~" H 3250 3150 50  0001 C CNN
 	1    3250 3150
@@
 F 0 "J6" H 1168 2725 50  0000 C CNN
 F 1 "COL5" H 1168 2816 50  0000 C CNN
-F 2 "Connector_PinHeader_2.54mm:PinHeader_1x06_P2.54mm_Vertical" H 1250 3150 50  0001 C CNN
+F 2 "Connector_JST:JST_XH_S6B-XH-A_1x06_P2.50mm_Horizontal" H 1250 3150 50  0001 C CNN
 F 3 "~" H 1250 3150 50  0001 C CNN
 	1    1250 3150
@@
 F 0 "J15" H 9168 4425 50  0000 C CNN
 F 1 "ROWS" H 9168 4516 50  0000 C CNN
-F 2 "Connector_PinHeader_2.54mm:PinHeader_1x06_P2.54mm_Vertical" H 9250 4850 50  0001 C CNN
+F 2 "Connector_JST:JST_XH_S6B-XH-A_1x06_P2.50mm_Horizontal" H 9250 4850 50  0001 C CNN
 F 3 "~" H 9250 4850 50  0001 C CNN
 	1    9250 4850

Commit message: Finished test board design
Parts:
- removed J1: COL0, Connector_JST:JST_XH_S6B-XH-A_1x06_P2.50mm_Horizontal, symbol Connector_Generic:Conn_01x05
- removed J10: COL9, Connector_JST:JST_XH_S6B-XH-A_1x06_P2.50mm_Horizontal, symbol Connector_Generic:Conn_01x05
- removed J11: COL10, Connector_JST:JST_XH_S6B-XH-A_1x06_P2.50mm_Horizontal, symbol Connector_Generic:Conn_01x04
- removed J12: COL11, Connector_JST:JST_XH_S6B-XH-A_1x06_P2.50mm_Horizontal, symbol Connector_Generic:Conn_01x05
- removed J13: COL12, Connector_JST:JST_XH_S6B-XH-A_1x06_P2.50mm_Horizontal, symbol Connector_Generic:Conn_01x05
- removed J14: COL13, Connector_JST:JST_XH_S6B-XH-A_1x06_P2.50mm_Horizontal, symbol Connector_Generic:Conn_01x05
- removed J15: ROWS, Connector_JST:JST_XH_S6B-XH-A_1x06_P2.50mm_Horizontal, symbol Connector_Generic:Conn_01x05
- removed J2: COL1, Connector_JST:JST_XH_S6B-XH-A_1x06_P2.50mm_Horizontal, symbol Connector_Generic:Conn_01x05
- removed J3: COL2, Connector_JST:JST_XH_S6B-XH-A_1x06_P2.50mm_Horizontal, symbol Connector_Generic:Conn_01x05
- removed J4: COL3, Connector_JST:JST_XH_S6B-XH-A_1x06_P2.50mm_Horizontal, symbol Connector_Generic:Conn_01x04
- removed J5: COL4, Connector_JST:JST_XH_S6B-XH-A_1x06_P2.50mm_Horizontal, symbol Connector_Generic:Conn_01x04
- removed J6: COL5, Connector_JST:JST_XH_S6B-XH-A_1x06_P2.50mm_Horizontal, symbol Connector_Generic:Conn_01x05
- removed J7: COL6, Connector_JST:JST_XH_S6B-XH-A_1x06_P2.50mm_Horizontal, symbol Connector_Generic:Conn_01x04
- removed J8: COL7, Connector_JST:JST_XH_S6B-XH-A_1x06_P2.50mm_Horizontal, symbol Connector_Generic:Conn_01x05
- removed J9: COL8, Connector_JST:JST_XH_S6B-XH-A_1x06_P2.50mm_Horizontal, symbol Connector_Generic:Conn_01x04
- added H1, H10, H11, H12, H2, H3, H4, H5, H6, H7, H8, H9: MountingHole_Pad, MountingHole:MountingHole_3.2mm_M3_DIN965_Pad_TopBottom, symbol Mechanical:MountingHole_Pad
- added J1: COL0, Connector_JST:JST_XH_S6B-XH-A_1x06_P2.50mm_Horizontal, symbol Connector_Generic:Conn_01x06
- added J10: COL9, Connector_JST:JST_XH_S6B-XH-A_1x06_P2.50mm_Horizontal, symbol Connector_Generic:Conn_01x06
- added J11: COL10, Connector_JST:JST_XH_S6B-XH-A_1x06_P2.50mm_Horizontal, symbol Connector_Generic:Conn_01x06
- added J12: COL11, Connector_JST:JST_XH_S6B-XH-A_1x06_P2.50mm_Horizontal, symbol Connector_Generic:Conn_01x06
- added J13: COL12, Connector_JST:JST_XH_S6B-XH-A_1x06_P2.50mm_Horizontal, symbol Connector_Generic:Conn_01x06
- added J14: COL13, Connector_JST:JST_XH_S6B-XH-A_1x06_P2.50mm_Horizontal, symbol Connector_Generic:Conn_01x06
- added J15: ROWS, Connector_JST:JST_XH_S6B-XH-A_1x06_P2.50mm_Horizontal, symbol Connector_Generic:Conn_01x06
- added J2: COL1, Connector_JST:JST_XH_S6B-XH-A_1x06_P2.50mm_Horizontal, symbol Connector_Generic:Conn_01x06
- added J3: COL2, Connector_JST:JST_XH_S6B-XH-A_1x06_P2.50mm_Horizontal, symbol Connector_Generic:Conn_01x06
- added J4: COL3, Connector_JST:JST_XH_S6B-XH-A_1x06_P2.50mm_Horizontal, symbol Connector_Generic:Conn_01x06
- added J5: COL4, Connector_JST:JST_XH_S6B-XH-A_1x06_P2.50mm_Horizontal, symbol Connector_Generic:Conn_01x06
- added J6: COL5, Connector_JST:JST_XH_S6B-XH-A_1x06_P2.50mm_Horizontal, symbol Connector_Generic:Conn_01x06
- added J7: COL6, Connector_JST:JST_XH_S6B-XH-A_1x06_P2.50mm_Horizontal, symbol Connector_Generic:Conn_01x06
- added J8: COL7, Connector_JST:JST_XH_S6B-XH-A_1x06_P2.50mm_Horizontal, symbol Connector_Generic:Conn_01x06
- added J9: COL8, Connector_JST:JST_XH_S6B-XH-A_1x06_P2.50mm_Horizontal, symbol Connector_Generic:Conn_01x06
- SW55: footprint Segment_Footprints:Segment_MX_1.00u_2.75u_PCB -> Segment_Footprints:Segment_MX_1.75u_2.75u_PCB
- SW56: footprint Segment_Footprints:Segment_MX_1.75u_PCB -> Segment_Footprints:Segment_MX_1.00u_PCB
Connections:
- net ROW0: now also J15.1 (Pin_1)
- net ROW1: now also J15.2 (Pin_2)
- net ROW2: now also J15.3 (Pin_3)
- net ROW3: now also J15.4 (Pin_4)
- net ROW4: now also J15.5 (Pin_5)
- net at SW57.1: now also J1.6 (Pin_6)
- net at SW43.1: now also J1.5 (Pin_5)
- net at SW29.1: now also J1.4 (Pin_4)
- net at SW15.1: now also J1.3 (Pin_3)
- net at SW1.1: now also J1.2 (Pin_2)
- net at SW58.1: now also J2.6 (Pin_6)
- net at SW44.1: now also J2.5 (Pin_5)
- net at SW30.1: now also J2.4 (Pin_4)
- net at SW16.1: now also J2.3 (Pin_3)
- net at SW2.1: now also J2.2 (Pin_2)
- net at SW59.1: now also J3.6 (Pin_6)
- net at SW45.1: now also J3.5 (Pin_5)
- net at SW31.1: now also J3.4 (Pin_4)
- net at SW17.1: now also J3.3 (Pin_3)
- net at SW3.1: now also J3.2 (Pin_2)
- net at SW46.1: now also J4.5 (Pin_5)
- net at SW32.1: now also J4.4 (Pin_4)
- net at SW18.1: now also J4.3 (Pin_3)
- net at SW4.1: now also J4.2 (Pin_2)
- net at SW47.1: now also J5.5 (Pin_5)
- net at SW33.1: now also J5.4 (Pin_4)
- net at SW19.1: now also J5.3 (Pin_3)
- net at SW5.1: now also J5.2 (Pin_2)
- net at SW60.1: now also J6.6 (Pin_6)
- net at SW48.1: now also J6.5 (Pin_5)
- net at SW34.1: now also J6.4 (Pin_4)
- net at SW20.1: now also J6.3 (Pin_3)
- net at SW6.1: now also J6.2 (Pin_2)
- net at SW49.1: now also J7.5 (Pin_5)
- net at SW35.1: now also J7.4 (Pin_4)
- net at SW21.1: now also J7.3 (Pin_3)
- net at SW7.1: now also J7.2 (Pin_2)
- net at SW61.1: now also J8.6 (Pin_6)
- net at SW50.1: now also J8.5 (Pin_5)
- net at SW36.1: now also J8.4 (Pin_4)
- net at SW22.1: now also J8.3 (Pin_3)
- net at SW8.1: now also J8.2 (Pin_2)
- net at SW51.1: now also J9.5 (Pin_5)
- net at SW37.1: now also J9.4 (Pin_4)
- net at SW23.1: now also J9.3 (Pin_3)
- net at SW9.1: now also J9.2 (Pin_2)
- net at SW62.1: now also J10.6 (Pin_6)
- net at SW52.1: now also J10.5 (Pin_5)
- net at SW38.1: now also J10.4 (Pin_4)
- net at SW24.1: now also J10.3 (Pin_3)
- net at SW10.1: now also J10.2 (Pin_2)
- net at SW53.1: now also J11.5 (Pin_5)
- net at SW39.1: now also J11.4 (Pin_4)
- net at SW25.1: now also J11.3 (Pin_3)
- net at SW11.1: now also J11.2 (Pin_2)
- net at SW63.1: now also J12.6 (Pin_6)
- net at SW54.1: now also J12.5 (Pin_5)
- net at SW40.1: now also J12.4 (Pin_4)
- net at SW26.1: now also J12.3 (Pin_3)
- net at SW12.1: now also J12.2 (Pin_2)
- net at SW64.1: now also J13.6 (Pin_6)
- net at SW55.1: now also J13.5 (Pin_5)
- net at SW41.1: now also J13.4 (Pin_4)
- net at SW27.1: now also J13.3 (Pin_3)
- net at SW13.1: now also J13.2 (Pin_2)
- net at SW65.1: now also J14.6 (Pin_6)
- net at SW56.1: now also J14.5 (Pin_5)
- net at SW42.1: now also J14.4 (Pin_4)
- net at SW28.1: now also J14.3 (Pin_3)
- net at SW14.1: now also J14.2 (Pin_2)
- new net GND: H1.1, H10.1, H11.1, H12.1, H2.1, H3.1, H4.1, H5.1, H6.1, H7.1, H8.1, H9.1
- no-connect marks 0 -> 20
Other:
- moved on the sheet: SW11, SW18, SW21, SW23, SW25, SW32, SW35, SW37, SW39, SW4, SW46, SW49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
