File: segment_TEST/segment_TEST.kicad_pcb (KiCad board)
At the start: 2 copper layers, 80 parts, among them J1 COL0, J10 COL9, J11 COL10, J12 COL11, J13 COL12, J14 COL13, J15 ROWS, J2 COL1, J3 COL2, J4 COL3, J5 COL4, J6 COL5, J7 COL6, J8 COL7, J9 COL8, SW1 SW_Push_45deg, SW10 SW_Push_45deg, SW11 SW_Push_45deg, SW12 SW_Push_45deg, SW13 SW_Push_45deg, SW14 SW_Push_45deg, SW15 SW_Push_45deg, SW16 SW_Push_45deg, SW17 SW_Push_45deg, SW18 SW_Push_45deg, SW19 SW_Push_45deg, SW2 SW_Push_45deg, SW20 SW_Push_45deg, SW21 SW_Push_45deg, SW22 SW_Push_45deg, SW23 SW_Push_45deg, SW24 SW_Push_45deg, SW25 SW_Push_45deg, SW26 SW_Push_45deg, SW27 SW_Push_45deg, SW28 SW_Push_45deg, SW29 SW_Push_45deg, SW3 SW_Push_45deg, SW30 SW_Push_45deg, SW31 SW_Push_45deg, SW32 SW_Push_45deg, SW33 SW_Push_45deg, SW34 SW_Push_45deg, SW35 SW_Push_45deg, SW36 SW_Push_45deg, SW37 SW_Push_45deg, SW38 SW_Push_45deg, SW39 SW_Push_45deg, SW4 SW_Push_45deg, SW40 SW_Push_45deg, SW41 SW_Push_45deg, SW42 SW_Push_45deg, SW43 SW_Push_45deg, SW44 SW_Push_45deg, SW45 SW_Push_45deg, SW46 SW_Push_45deg, SW47 SW_Push_45deg, SW48 SW_Push_45deg, SW49 SW_Push_45deg, SW5 SW_Push_45deg, SW50 SW_Push_45deg, SW51 SW_Push_45deg, SW52 SW_Push_45deg, SW53 SW_Push_45deg, SW54 SW_Push_45deg, SW55 SW_Push_45deg, SW56 SW_Push_45deg, SW57 SW_Push_45deg, SW58 SW_Push_45deg, SW59 SW_Push_45deg, SW6 SW_Push_45deg, SW60 SW_Push_45deg, SW61 SW_Push_45deg, SW62 SW_Push_45deg, SW63 SW_Push_45deg, SW64 SW_Push_45deg, SW65 SW_Push_45deg, SW7 SW_Push_45deg, SW8 SW_Push_45deg, SW9 SW_Push_45deg

Commit message: Completed test board layout; implementing option footprints
Parts:
- SW1, SW10, SW11, SW12, SW13, SW16, SW17, SW18, SW19, SW2, SW20, SW21, SW22, SW23, SW24, SW25, SW26, SW27, SW28, SW3, SW30, SW31, SW32, SW33, SW34, SW35, SW36, SW37, SW38, SW39, SW4, SW40, SW44, SW45, SW46, SW47, SW48, SW49, SW5, SW50, SW51, SW52, SW53, SW54, SW56, SW58, SW6, SW64, SW7, SW8, SW9: footprint Button_Switch_Keyboard:SW_Cherry_MX_1.00u_PCB -> Segment_Footprints:Segment_MX_1.00u_PCB
- SW14: footprint Button_Switch_Keyboard:SW_Cherry_MX_1.00u_PCB -> Segment_Footprints:Segment_MX_1.00u_2.00u_PCB
- SW15, SW42, SW57, SW59, SW63, SW65: footprint Button_Switch_Keyboard:SW_Cherry_MX_1.50u_PCB -> Segment_Footprints:Segment_MX_1.50u_PCB
- SW29, SW55: footprint Button_Switch_Keyboard:SW_Cherry_MX_1.75u_PCB -> Segment_Footprints:Segment_MX_1.75u_PCB
- SW41: footprint Button_Switch_Keyboard:SW_Cherry_MX_2.25u_PCB -> Segment_Footprints:Segment_MX_2.25u_PCB
- SW43: footprint Button_Switch_Keyboard:SW_Cherry_MX_1.25u_PCB -> Segment_Footprints:Segment_MX_1.25u_2.25u_PCB
- SW60, SW62: footprint Button_Switch_Keyboard:SW_Cherry_MX_2.75u_PCB -> Segment_Footprints:Segment_MX_2.75u_PCB
- SW61: footprint Button_Switch_Keyboard:SW_Cherry_MX_1.50u_PCB -> Segment_Footprints:Segment_MX_7.00u_PCB
- moved SW10 19.1 mm to (234.9, 88.9)
- moved SW11 19.1 mm to (254.0, 88.9)
- moved SW12 19.1 mm to (273.1, 88.9)
- moved SW14 19.1 mm to (311.1, 88.9)
- moved SW17 19.1 mm to (111.1, 108.0)
- moved SW19 19.1 mm to (149.2, 108.0)
- moved SW21 19.1 mm to (187.3, 108.0)
- moved SW22 19.1 mm to (206.4, 108.0)
- moved SW25 19.1 mm to (263.5, 108.0)
- moved SW26 19.1 mm to (282.6, 108.0)
- moved SW27 19.1 mm to (301.6, 108.0)
- moved SW28 19.1 mm to (330.2, 88.9)
- moved SW3 19.1 mm to (101.6, 88.9)
- moved SW32 19.1 mm to (134.9, 127.0)
- moved SW34 19.1 mm to (173.0, 127.0)
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Other:
- board outline added: 285.8 x 104.1 mm

Commit message: Layout mostly complete for test board
Parts:
- removed J1: COL0, Connector_PinHeader_2.54mm:PinHeader_1x05_P2.54mm_Vertical
- added COL0: COL0, Connector_PinHeader_2.54mm:PinHeader_1x06_P2.54mm_Vertical, F.Cu at (69.8, 76.2)
- J10, J12, J13, J14, J15, J2, J3, J6, J8: footprint Connector_PinHeader_2.54mm:PinHeader_1x05_P2.54mm_Vertical -> Connector_PinHeader_2.54mm:PinHeader_1x06_P2.54mm_Vertical
- J11, J4, J5, J7, J9: footprint Connector_PinHeader_2.54mm:PinHeader_1x04_P2.54mm_Vertical -> Connector_PinHeader_2.54mm:PinHeader_1x06_P2.54mm_Vertical
- SW29: footprint Segment_Footprints:Segment_MX_1.75u_PCB -> Segment_Footprints:Segment_MX_1.25u_1.75u_PCB
- SW41: footprint Segment_Footprints:Segment_MX_2.25u_PCB -> Segment_Footprints:Segment_MX_1.00u_2.25u_PCB
- SW42: footprint Segment_Footprints:Segment_MX_1.50u_PCB -> Segment_Footprints:Segment_MX_1.50u_ISO_PCB
- SW55: footprint Segment_Footprints:Segment_MX_1.75u_PCB -> Segment_Footprints:Segment_MX_1.00u_2.75u_PCB
- SW56: footprint Segment_Footprints:Segment_MX_1.00u_PCB -> Segment_Footprints:Segment_MX_1.75u_PCB
- moved SW55 26.2 mm to (296.9, 146.1)
- moved SW56 26.2 mm to (323.1, 146.1)
- moved SW41 11.9 mm to (306.4, 127.0)
- moved J10 11.5 mm to (241.3, 76.2), turned to 270 degrees
- moved J13 11.5 mm to (298.4, 76.2), turned to 270 degrees
- moved J14 11.5 mm to (317.5, 76.2), turned to 270 degrees
- moved J15 11.5 mm to (336.6, 76.2), turned to 270 degrees
- moved J2 11.5 mm to (88.9, 76.2), turned to 270 degrees
- moved J3 11.5 mm to (108.0, 76.2), turned to 270 degrees
- moved J6 11.5 mm to (165.1, 76.2), turned to 270 degrees
- moved J8 11.5 mm to (203.2, 76.2), turned to 270 degrees
- moved J12 11.5 mm to (279.4, 76.2), turned to 270 degrees
- moved J11 10.2 mm to (260.4, 76.2), turned to 270 degrees
- moved J5 10.2 mm to (146.1, 76.2), turned to 270 degrees
- moved J4 10.2 mm to (127.0, 76.2), turned to 270 degrees
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
Commit message: Added JST-XH connectors to test board
Parts:
- removed J2: COL1, Connector_PinHeader_2.54mm:PinHeader_1x06_P2.54mm_Vertical
- removed J3: COL2, Connector_PinHeader_2.54mm:PinHeader_1x06_P2.54mm_Vertical
- removed J4: COL3, Connector_PinHeader_2.54mm:PinHeader_1x06_P2.54mm_Vertical
- added COL1: COL1, Connector_JST:JST_XH_S6B-XH-A_1x06_P2.50mm_Horizontal, F.Cu at (88.9, 76.2)
- added COL2: COL2, Connector_JST:JST_XH_S6B-XH-A_1x06_P2.50mm_Horizontal, F.Cu at (108.0, 76.2)
- added COL3: COL3, Connector_JST:JST_XH_S6B-XH-A_1x06_P2.50mm_Horizontal, F.Cu at (127.0, 76.2)
- COL0, J10, J11, J12, J13, J14, J15, J5, J6, J7, J8, J9: footprint Connector_PinHeader_2.54mm:PinHeader_1x06_P2.54mm_Vertical -> Connector_JST:JST_XH_S6B-XH-A_1x06_P2.50mm_Horizontal
- turned COL0 to 180 degrees
- turned J10 to 180 degrees
- turned J11 to 180 degrees
- turned J12 to 180 degrees
- turned J13 to 180 degrees
- turned J14 to 180 degrees
- turned J15 to 180 degrees
- turned J5 to 180 degrees
- turned J6 to 180 degrees
- turned J7 to 180 degrees
- turned J8 to 180 degrees
- turned J9 to 180 degrees
Other:
- board size 285.8 x 104.1 mm -> 285.8 x 110.5 mm

Commit message: Added mounting holes to test board
Parts:
- removed J10: COL9, Connector_JST:JST_XH_S6B-XH-A_1x06_P2.50mm_Horizontal
- removed J11: COL10, Connector_JST:JST_XH_S6B-XH-A_1x06_P2.50mm_Horizontal
- removed J12: COL11, Connector_JST:JST_XH_S6B-XH-A_1x06_P2.50mm_Horizontal
- removed J13: COL12, Connector_JST:JST_XH_S6B-XH-A_1x06_P2.50mm_Horizontal
- removed J14: COL13, Connector_JST:JST_XH_S6B-XH-A_1x06_P2.50mm_Horizontal
- removed J15: ROWS, Connector_JST:JST_XH_S6B-XH-A_1x06_P2.50mm_Horizontal
- removed J5: COL4, Connector_JST:JST_XH_S6B-XH-A_1x06_P2.50mm_Horizontal
- removed J6: COL5, Connector_JST:JST_XH_S6B-XH-A_1x06_P2.50mm_Horizontal
- removed J7: COL6, Connector_JST:JST_XH_S6B-XH-A_1x06_P2.50mm_Horizontal
- removed J8: COL7, Connector_JST:JST_XH_S6B-XH-A_1x06_P2.50mm_Horizontal
- removed J9: COL8, Connector_JST:JST_XH_S6B-XH-A_1x06_P2.50mm_Horizontal
- added COL10: COL10, Connector_JST:JST_XH_S6B-XH-A_1x06_P2.50mm_Horizontal, F.Cu at (260.2, 75.6)
- added COL11: COL11, Connector_JST:JST_XH_S6B-XH-A_1x06_P2.50mm_Horizontal, F.Cu at (279.3, 75.6)
- added COL12: COL12, Connector_JST:JST_XH_S6B-XH-A_1x06_P2.50mm_Horizontal, F.Cu at (298.4, 75.6)
- added COL13: COL13, Connector_JST:JST_XH_S6B-XH-A_1x06_P2.50mm_Horizontal, F.Cu at (317.4, 75.6)
- added COL4: COL4, Connector_JST:JST_XH_S6B-XH-A_1x06_P2.50mm_Horizontal, F.Cu at (145.9, 75.6)
- added COL5: COL5, Connector_JST:JST_XH_S6B-XH-A_1x06_P2.50mm_Horizontal, F.Cu at (165.0, 75.6)
- added COL6: COL6, Connector_JST:JST_XH_S6B-XH-A_1x06_P2.50mm_Horizontal, F.Cu at (184.1, 75.6)
- added COL7: COL7, Connector_JST:JST_XH_S6B-XH-A_1x06_P2.50mm_Horizontal, F.Cu at (203.1, 75.6)
- added COL8: COL8, Connector_JST:JST_XH_S6B-XH-A_1x06_P2.50mm_Horizontal, F.Cu at (222.2, 75.6)
- added COL9: COL9, Connector_JST:JST_XH_S6B-XH-A_1x06_P2.50mm_Horizontal, F.Cu at (241.2, 75.6)
- added REF**: MountingHole_3.2mm_M3_DIN965_Pad_TopBottom, MountingHole:MountingHole_3.2mm_M3_DIN965_Pad_TopBottom, F.Cu at (215.9, 99.1)
- added REF**: MountingHole_3.2mm_M3_DIN965_Pad_TopBottom, MountingHole:MountingHole_3.2mm_M3_DIN965_Pad_TopBottom, F.Cu at (50.8, 171.4)
- added REF**: MountingHole_3.2mm_M3_DIN965_Pad_TopBottom, MountingHole:MountingHole_3.2mm_M3_DIN965_Pad_TopBottom, F.Cu at (342.9, 171.4)
- added REF**: MountingHole_3.2mm_M3_DIN965_Pad_TopBottom, MountingHole:MountingHole_3.2mm_M3_DIN965_Pad_TopBottom, F.Cu at (342.9, 68.6)
- added REF**: MountingHole_3.2mm_M3_DIN965_Pad_TopBottom, MountingHole:MountingHole_3.2mm_M3_DIN965_Pad_TopBottom, F.Cu at (215.9, 156.2)
- added REF**: MountingHole_3.2mm_M3_DIN965_Pad_TopBottom, MountingHole:MountingHole_3.2mm_M3_DIN965_Pad_TopBottom, F.Cu at (177.8, 99.1)
- added REF**: MountingHole_3.2mm_M3_DIN965_Pad_TopBottom, MountingHole:MountingHole_3.2mm_M3_DIN965_Pad_TopBottom, F.Cu at (177.8, 156.2)
- added REF**: MountingHole_3.2mm_M3_DIN965_Pad_TopBottom, MountingHole:MountingHole_3.2mm_M3_DIN965_Pad_TopBottom, F.Cu at (101.6, 99.1)
- added REF**: MountingHole_3.2mm_M3_DIN965_Pad_TopBottom, MountingHole:MountingHole_3.2mm_M3_DIN965_Pad_TopBottom, F.Cu at (292.1, 99.1)
- added REF**: MountingHole_3.2mm_M3_DIN965_Pad_TopBottom, MountingHole:MountingHole_3.2mm_M3_DIN965_Pad_TopBottom, F.Cu at (292.1, 156.2)
- added REF**: MountingHole_3.2mm_M3_DIN965_Pad_TopBottom, MountingHole:MountingHole_3.2mm_M3_DIN965_Pad_TopBottom, F.Cu at (101.6, 156.2)
- added REF**: MountingHole_3.2mm_M3_DIN965_Pad_TopBottom, MountingHole:MountingHole_3.2mm_M3_DIN965_Pad_TopBottom, F.Cu at (50.8, 68.6)
- added ROWS: ROWS, Connector_JST:JST_XH_S6B-XH-A_1x06_P2.50mm_Horizontal, F.Cu at (336.4, 75.6)
- moved COL1 0.64 mm to (88.8, 75.6)
- moved COL2 0.64 mm to (107.8, 75.6)
- moved COL0 0.64 mm to (69.8, 75.6)
- moved COL3 0.64 mm to (126.9, 75.6)
Other:
- board size 285.8 x 110.5 mm -> 298.4 x 109.2 mm
- net class Through Hole added: clearance 0.3, trace_width 0.3, via_dia 0.8, via_drill 0.4

Commit message: Finished test board design
Parts:
- removed REF** (x12): MountingHole_3.2mm_M3_DIN965_Pad_TopBottom, MountingHole:MountingHole_3.2mm_M3_DIN965_Pad_TopBottom
- added H1: MountingHole_Pad, MountingHole:MountingHole_3.2mm_M3_DIN965_Pad_TopBottom, F.Cu at (50.8, 68.6)
- added H10: MountingHole_Pad, MountingHole:MountingHole_3.2mm_M3_DIN965_Pad_TopBottom, F.Cu at (215.9, 156.2)
- added H11: MountingHole_Pad, MountingHole:MountingHole_3.2mm_M3_DIN965_Pad_TopBottom, F.Cu at (292.1, 156.2)
- added H12: MountingHole_Pad, MountingHole:MountingHole_3.2mm_M3_DIN965_Pad_TopBottom, F.Cu at (342.9, 171.4)
- added H2: MountingHole_Pad, MountingHole:MountingHole_3.2mm_M3_DIN965_Pad_TopBottom, F.Cu at (101.6, 99.1)
- added H3: MountingHole_Pad, MountingHole:MountingHole_3.2mm_M3_DIN965_Pad_TopBottom, F.Cu at (177.8, 99.1)
- added H4: MountingHole_Pad, MountingHole:MountingHole_3.2mm_M3_DIN965_Pad_TopBottom, F.Cu at (215.9, 99.1)
- added H5: MountingHole_Pad, MountingHole:MountingHole_3.2mm_M3_DIN965_Pad_TopBottom, F.Cu at (292.1, 99.1)
- added H6: MountingHole_Pad, MountingHole:MountingHole_3.2mm_M3_DIN965_Pad_TopBottom, F.Cu at (342.9, 68.6)
- added H7: MountingHole_Pad, MountingHole:MountingHole_3.2mm_M3_DIN965_Pad_TopBottom, F.Cu at (50.8, 171.4)
- added H8: MountingHole_Pad, MountingHole:MountingHole_3.2mm_M3_DIN965_Pad_TopBottom, F.Cu at (101.6, 156.2)
- added H9: MountingHole_Pad, MountingHole:MountingHole_3.2mm_M3_DIN965_Pad_TopBottom, F.Cu at (177.8, 156.2)
- SW55: footprint Segment_Footprints:Segment_MX_1.00u_2.75u_PCB -> Segment_Footprints:Segment_MX_1.75u_2.75u_PCB
- SW56: footprint Segment_Footprints:Segment_MX_1.75u_PCB -> Segment_Footprints:Segment_MX_1.00u_PCB
- moved SW55 7.14 mm to (304.0, 146.1)
- moved SW56 7.14 mm to (330.2, 146.1)
Connections:
- COL0 pad 6: (no net) -> Net-(J1-Pad6)
- COL1 pad 6: (no net) -> Net-(J2-Pad6)
- COL10 pad 5: (no net) -> Net-(J11-Pad5)
- COL10 pad 6: (no net) -> Net-(J11-Pad6)
- COL11 pad 6: (no net) -> Net-(J12-Pad6)
- COL12 pad 6: (no net) -> Net-(J13-Pad6)
- COL13 pad 6: (no net) -> Net-(J14-Pad6)
- COL2 pad 6: (no net) -> Net-(J3-Pad6)
- COL3 pad 5: (no net) -> Net-(J4-Pad5)
- COL3 pad 6: (no net) -> Net-(J4-Pad6)
- COL4 pad 5: (no net) -> Net-(J5-Pad5)
- COL4 pad 6: (no net) -> Net-(J5-Pad6)
- COL5 pad 6: (no net) -> Net-(J6-Pad6)
- COL6 pad 5: (no net) -> Net-(J7-Pad5)
- COL6 pad 6: (no net) -> Net-(J7-Pad6)
- COL7 pad 6: (no net) -> Net-(J8-Pad6)
- COL8 pad 5: (no net) -> Net-(J9-Pad5)
- COL8 pad 6: (no net) -> Net-(J9-Pad6)
- COL9 pad 6: (no net) -> Net-(J10-Pad6)
- ROWS pad 6: (no net) -> Net-(J15-Pad6)
- SW1 pad 1: Net-(J1-Pad5) -> Net-(J1-Pad2)
- SW10 pad 1: Net-(J10-Pad5) -> Net-(J10-Pad2)
- SW11 pad 1: Net-(J11-Pad4) -> Net-(J11-Pad2)
- SW12 pad 1: Net-(J12-Pad5) -> Net-(J12-Pad2)
- SW13 pad 1: Net-(J13-Pad5) -> Net-(J13-Pad2)
- SW14 pad 1: Net-(J14-Pad5) -> Net-(J14-Pad2)
- SW15 pad 1: Net-(J1-Pad4) -> Net-(J1-Pad3)
- SW16 pad 1: Net-(J2-Pad4) -> Net-(J2-Pad3)
- SW17 pad 1: Net-(J3-Pad4) -> Net-(J3-Pad3)
- SW2 pad 1: Net-(J2-Pad5) -> Net-(J2-Pad2)
- SW20 pad 1: Net-(J6-Pad4) -> Net-(J6-Pad3)
- SW22 pad 1: Net-(J8-Pad4) -> Net-(J8-Pad3)
- SW24 pad 1: Net-(J10-Pad4) -> Net-(J10-Pad3)
- SW26 pad 1: Net-(J12-Pad4) -> Net-(J12-Pad3)
- SW27 pad 1: Net-(J13-Pad4) -> Net-(J13-Pad3)
- SW28 pad 1: Net-(J14-Pad4) -> Net-(J14-Pad3)
- SW29 pad 1: Net-(J1-Pad3) -> Net-(J1-Pad4)
- SW3 pad 1: Net-(J3-Pad5) -> Net-(J3-Pad2)
- SW30 pad 1: Net-(J2-Pad3) -> Net-(J2-Pad4)
- SW31 pad 1: Net-(J3-Pad3) -> Net-(J3-Pad4)
- SW32 pad 1: Net-(J4-Pad2) -> Net-(J4-Pad4)
- SW33 pad 1: Net-(J5-Pad2) -> Net-(J5-Pad4)
- SW34 pad 1: Net-(J6-Pad3) -> Net-(J6-Pad4)
- SW35 pad 1: Net-(J7-Pad2) -> Net-(J7-Pad4)
- SW36 pad 1: Net-(J8-Pad3) -> Net-(J8-Pad4)
- SW37 pad 1: Net-(J9-Pad2) -> Net-(J9-Pad4)
- SW38 pad 1: Net-(J10-Pad3) -> Net-(J10-Pad4)
- SW39 pad 1: Net-(J11-Pad2) -> Net-(J11-Pad4)
- SW4 pad 1: Net-(J4-Pad4) -> Net-(J4-Pad2)
- SW40 pad 1: Net-(J12-Pad3) -> Net-(J12-Pad4)
- SW41 pad 1: Net-(J13-Pad3) -> Net-(J13-Pad4)
- SW42 pad 1: Net-(J14-Pad3) -> Net-(J14-Pad4)
- SW43 pad 1: Net-(J1-Pad2) -> Net-(J1-Pad5)
- SW44 pad 1: Net-(J2-Pad2) -> Net-(J2-Pad5)
- SW45 pad 1: Net-(J3-Pad2) -> Net-(J3-Pad5)
- SW46 pad 1: Net-(J4-Pad1) -> Net-(J4-Pad5)
- SW47 pad 1: Net-(J5-Pad1) -> Net-(J5-Pad5)
- SW48 pad 1: Net-(J6-Pad2) -> Net-(J6-Pad5)
- SW49 pad 1: Net-(J7-Pad1) -> Net-(J7-Pad5)
- SW5 pad 1: Net-(J5-Pad4) -> Net-(J5-Pad2)
- SW50 pad 1: Net-(J8-Pad2) -> Net-(J8-Pad5)
- SW51 pad 1: Net-(J9-Pad1) -> Net-(J9-Pad5)
- SW52 pad 1: Net-(J10-Pad2) -> Net-(J10-Pad5)
- SW53 pad 1: Net-(J11-Pad1) -> Net-(J11-Pad5)
- SW54 pad 1: Net-(J12-Pad2) -> Net-(J12-Pad5)
- SW55 pad 1: Net-(J13-Pad2) -> Net-(J13-Pad5)
- SW56 pad 1: Net-(J14-Pad2) -> Net-(J14-Pad5)
- SW57 pad 1: Net-(J1-Pad1) -> Net-(J1-Pad6)
- SW58 pad 1: Net-(J2-Pad1) -> Net-(J2-Pad6)
- SW59 pad 1: Net-(J3-Pad1) -> Net-(J3-Pad6)
- SW6 pad 1: Net-(J6-Pad5) -> Net-(J6-Pad2)
- SW60 pad 1: Net-(J6-Pad1) -> Net-(J6-Pad6)
- SW61 pad 1: Net-(J8-Pad1) -> Net-(J8-Pad6)
- SW62 pad 1: Net-(J10-Pad1) -> Net-(J10-Pad6)
- SW63 pad 1: Net-(J12-Pad1) -> Net-(J12-Pad6)
- SW64 pad 1: Net-(J13-Pad1) -> Net-(J13-Pad6)
- SW65 pad 1: Net-(J14-Pad1) -> Net-(J14-Pad6)
- SW7 pad 1: Net-(J7-Pad4) -> Net-(J7-Pad2)
- SW8 pad 1: Net-(J8-Pad5) -> Net-(J8-Pad2)
- SW9 pad 1: Net-(J9-Pad4) -> Net-(J9-Pad2)
Routing:
- net ROW0: track 0.00 -> 346.7 mm
- net ROW1: track 0.00 -> 333.1 mm
- net ROW2: track 0.00 -> 317.6 mm
- net ROW3: track 0.00 -> 283.5 mm
- net ROW4: track 0.00 -> 266.9 mm
- net Net-(J14-Pad6): track 0.00 -> 133.0 mm
- net Net-(J14-Pad5): track 0.00 -> 107.6 mm
- net Net-(J3-Pad6): track 0.00 -> 102.5 mm
- net Net-(J2-Pad6): track 0.00 -> 101.8 mm
- net Net-(J6-Pad6): track 0.00 -> 99.3 mm
- net Net-(J12-Pad6): track 0.00 -> 98.5 mm
- net Net-(J8-Pad6): track 0.00 -> 98.3 mm
- net Net-(J10-Pad6): track 0.00 -> 97.6 mm
- net Net-(J13-Pad6): track 0.00 -> 94.6 mm
- net Net-(J1-Pad6): track 0.00 -> 92.8 mm
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- added copper zone on B.Cu, net (none)
- added copper zone on B.Cu, net GND
- added copper zone on F.Cu, net GND
Other:
- net class Default: clearance 0.2 -> 0.381; trace_width 0.25 -> 0.381
- net class Rows added: clearance 0.381, trace_width 0.508, via_dia 0.8, via_drill 0.4
- net class Through Hole: clearance 0.3 -> 0.381; trace_width 0.3 -> 0.381; via_dia 0.8 -> 1.2; via_drill 0.4 -> 0.6
- rule trace_clearance: 0.2 -> 0.381
- board text added: "2020-3"
- board text added: "COL0"
- board text added: "COL1"
- board text added: "COL10"
- board text added: "COL11"
- board text added: "COL12"
- board text added: "COL13"
- board text added: "COL2"
- board text added: "COL3"
- board text added: "COL4"
- board text added: "COL5"
- board text added: "COL6"
- board text added: "COL7"
- board text added: "COL8"
- board text added: "COL9"
- board text added: "DEVELOPMENT KEY MATRIX"
- board text added: "R-1.0.0"
- board text added: "R0"
- board text added: "R1"
- board text added: "R2"
- board text added: "R3"
- board text added: "R4"
- board text added: "ROWS"
- board text added: "SEGMENT-60"

Commit message: Minor tweak to test board
Routing:
- net Net-(J13-Pad6): track 94.6 -> 93.4 mm
- net Net-(J13-Pad5): track 86.4 -> 85.4 mm

Commit message: Updated test board
Routing:
- net Net-(J1-Pad6): track 92.8 -> 91.6 mm
- net Net-(J1-Pad5): track 82.7 -> 81.5 mm
Other:
- board text added: "2021-3"
- board text added: "R-1.0.1"
- board text removed: "2020-3"
- board text removed: "R-1.0.0"
