File: segment_TEST/segment_TEST.kicad_pcb (KiCad board)
At the start: 2 copper layers, 298.4 x 109.2 mm, 92 parts, among them SW1 SW_Push_45deg, SW10 SW_Push_45deg, SW11 SW_Push_45deg, SW12 SW_Push_45deg, SW13 SW_Push_45deg, SW14 SW_Push_45deg, SW15 SW_Push_45deg, SW16 SW_Push_45deg, SW17 SW_Push_45deg, SW18 SW_Push_45deg, SW19 SW_Push_45deg, SW2 SW_Push_45deg, SW20 SW_Push_45deg, SW21 SW_Push_45deg, SW22 SW_Push_45deg, SW23 SW_Push_45deg, SW24 SW_Push_45deg, SW25 SW_Push_45deg, SW26 SW_Push_45deg, SW27 SW_Push_45deg, SW28 SW_Push_45deg, SW29 SW_Push_45deg, SW3 SW_Push_45deg, SW30 SW_Push_45deg, SW31 SW_Push_45deg, SW32 SW_Push_45deg, SW33 SW_Push_45deg, SW34 SW_Push_45deg, SW35 SW_Push_45deg, SW36 SW_Push_45deg, SW37 SW_Push_45deg, SW38 SW_Push_45deg, SW39 SW_Push_45deg, SW4 SW_Push_45deg, SW40 SW_Push_45deg, SW41 SW_Push_45deg, SW42 SW_Push_45deg, SW43 SW_Push_45deg, SW44 SW_Push_45deg, SW45 SW_Push_45deg, SW46 SW_Push_45deg, SW47 SW_Push_45deg, SW48 SW_Push_45deg, SW49 SW_Push_45deg, SW5 SW_Push_45deg, SW50 SW_Push_45deg, SW51 SW_Push_45deg, SW52 SW_Push_45deg, SW53 SW_Push_45deg, SW54 SW_Push_45deg, SW55 SW_Push_45deg, SW56 SW_Push_45deg, SW57 SW_Push_45deg, SW58 SW_Push_45deg, SW59 SW_Push_45deg, SW6 SW_Push_45deg, SW60 SW_Push_45deg, SW61 SW_Push_45deg, SW62 SW_Push_45deg, SW63 SW_Push_45deg, SW64 SW_Push_45deg, SW65 SW_Push_45deg, SW7 SW_Push_45deg, SW8 SW_Push_45deg, SW9 SW_Push_45deg

Commit message: Added test board dimensions
Changed lines of the file:
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@@
-(kicad_pcb (version 20171130) (host pcbnew 5.1.9)
+(kicad_pcb (version 20171130) (host pcbnew 5.1.10)
   (general
     (thickness 1.6)
-    (drawings 217)
+    (drawings 229)
     (tracks 6036)
     (zones 0)
@@
     (46 B.CrtYd user)
     (47 F.CrtYd user)
-    (48 B.Fab user)
-    (49 F.Fab user)
+    (48 B.Fab user hide)
+    (49 F.Fab user hide)
   )
   (setup
@@
     (visible_elements FFFFFF7F)
     (pcbplotparams
-      (layerselection 0x010f0_ffffffff)
+      (layerselection 0x011f0_ffffffff)
       (usegerberextensions false)
       (usegerberattributes true)
@@
       (padsonsilk false)
       (subtractmaskfromsilk false)
-      (outputformat 1)
+      (outputformat 4)
       (mirror false)
       (drillshape 0)
@@
     (pad "" np_thru_hole circle (at -5.08 0) (size 1.7 1.7) (drill 1.7) (layers *.Cu *.Mask))
   )
+  (dimension 33.655 (width 0.15) (layer Dwgs.User)
+    (gr_text "1.3250 in" (at 351.185 82.2325 90) (layer Dwgs.User)
+      (effects (font (size 1 1) (thickness 0.15)))
+    )
+    (feature1 (pts (xy 292.1 65.405) (xy 350.471421 65.405)))
+    (feature2 (pts (xy 292.1 99.06) (xy 350.471421 99.06)))
+    (crossbar (pts (xy 349.885 99.06) (xy 349.885 65.405)))
+    (arrow1a (pts (xy 349.885 65.405) (xy 350.471421 66.531504)))
+    (arrow1b (pts (xy 349.885 65.405) (xy 349.298579 66.531504)))
+    (arrow2a (pts (xy 349.885 99.06) (xy 350.471421 97.933496)))
+    (arrow2b (pts (xy 349.885 99.06) (xy 349.298579 97.933496)))
+  )
+  (dimension 57.15 (width 0.15) (layer Dwgs.User)
+    (gr_text "2.2500 in" (at 351.185 127.635 90) (layer Dwgs.User)
+      (effects (font (size 1 1) (thickness 0.15)))
+    )
+    (feature1 (pts (xy 292.1 99.06) (xy 350.471421 99.06)))
+    (feature2 (pts (xy 292.1 156.21) (xy 350.471421 156.21)))
+    (crossbar (pts (xy 349.885 156.21) (xy 349.885 99.06)))
+    (arrow1a (pts (xy 349.885 99.06) (xy 350.471421 100.186504)))
+    (arrow1b (pts (xy 349.885 99.06) (xy 349.298579 100.186504)))
+    (arrow2a (pts (xy 349.885 156.21) (xy 350.471421 155.083496)))
+    (arrow2b (pts (xy 349.885 156.21) (xy 349.298579 155.083496)))
+  )
+  (dimension 109.22 (width 0.15) (layer Dwgs.User)
+    (gr_text "4.3000 in" (at 38.705 120.015 90) (layer Dwgs.User)
+      (effects (font (size 1 1) (thickness 0.15)))
+    )
+    (feature1 (pts (xy 50.8 65.405) (xy 39.418579 65.405)))
+    (feature2 (pts (xy 50.8 174.625) (xy 39.418579 174.625)))
+    (crossbar (pts (xy 40.005 174.625) (xy 40.005 65.405)))
+    (arrow1a (pts (xy 40.005 65.405) (xy 40.591421 66.531504)))
+    (arrow1b (pts (xy 40.005 65.405) (xy 39.418579 66.531504)))
+    (arrow2a (pts (xy 40.005 174.625) (xy 40.591421 173.498496)))
+    (arrow2b (pts (xy 40.005 174.625) (xy 39.418579 173.498496)))
+  )
+  (dimension 102.87 (width 0.15) (layer Dwgs.User)
+    (gr_text "4.0500 in" (at 42.515 120.015 90) (layer Dwgs.User)
+      (effects (font (size 1 1) (thickness 0.15)))
+    )
+    (feature1 (pts (xy 50.8 68.58) (xy 43.228579 68.58)))
+    (feature2 (pts (xy 50.8 171.45) (xy 43.228579 171.45)))
+    (crossbar (pts (xy 43.815 171.45) (xy 43.815 68.58)))
+    (arrow1a (pts (xy 43.815 68.58) (xy 44.401421 69.706504)))
+    (arrow1b (pts (xy 43.815 68.58) (xy 43.228579 69.706504)))
+    (arrow2a (pts (xy 43.815 171.45) (xy 44.401421 170.323496)))
+    (arrow2b (pts (xy 43.815 171.45) (xy 43.228579 170.323496)))
+  )
+  (dimension 18.415 (width 0.15) (layer Dwgs.User)
+    (gr_text "0.7250 in" (at 351.185 165.4175 270) (layer Dwgs.User)
+      (effects (font (size 1 1) (thickness 0.15)))
+    )
+    (feature1 (pts (xy 292.1 174.625) (xy 350.471421 174.625)))
+    (feature2 (pts (xy 292.1 156.21) (xy 350.471421 156.21)))
+    (crossbar (pts (xy 349.885 156.21) (xy 349.885 174.625)))
+    (arrow1a (pts (xy 349.885 174.625) (xy 349.298579 173.498496)))
+    (arrow1b (pts (xy 349.885 174.625) (xy 350.471421 173.498496)))
+    (arrow2a (pts (xy 349.885 156.21) (xy 349.298579 157.336504)))
+    (arrow2b (pts (xy 349.885 156.21) (xy 350.471421 157.336504)))
+  )
+  (dimension 53.975 (width 0.15) (layer Dwgs.User)
+    (gr_text "2.1250 in" (at 74.6125 179.735) (layer Dwgs.User)
+      (effects (font (size 1 1) (thickness 0.15)))
+    )
+    (feature1 (pts (xy 47.625 156.21) (xy 47.625 179.021421)))
+    (feature2 (pts (xy 101.6 156.21) (xy 101.6 179.021421)))
+    (crossbar (pts (xy 101.6 178.435) (xy 47.625 178.435)))
+    (arrow1a (pts (xy 47.625 178.435) (xy 48.751504 177.848579)))
+    (arrow1b (pts (xy 47.625 178.435) (xy 48.751504 179.021421)))
+    (arrow2a (pts (xy 101.6 178.435) (xy 100.473496 177.848579)))
+    (arrow2b (pts (xy 101.6 178.435) (xy 100.473496 179.021421)))
+  )
+  (dimension 53.975 (width 0.15) (layer Dwgs.User)
+    (gr_text "2.1250 in" (at 319.0875 179.735) (layer Dwgs.User)
+      (effects (font (size 1 1) (thickness 0.15)))
+    )
+    (feature1 (pts (xy 346.075 156.21) (xy 346.075 179.021421)))
+    (feature2 (pts (xy 292.1 156.21) (xy 292.1 179.021421)))
+    (crossbar (pts (xy 292.1 178.435) (xy 346.075 178.435)))
+    (arrow1a (pts (xy 346.075 178.435) (xy 344.948496 179.021421)))
+    (arrow1b (pts (xy 346.075 178.435) (xy 344.948496 177.848579)))
+    (arrow2a (pts (xy 292.1 178.435) (xy 293.226504 179.021421)))
+    (arrow2b (pts (xy 292.1 178.435) (xy 293.226504 177.848579)))
+  )
+  (dimension 76.2 (width 0.15) (layer Dwgs.User)
+    (gr_text "3.0000 in" (at 254 179.734999) (layer Dwgs.User)
+      (effects (font (size 1 1) (thickness 0.15)))
+    )
+    (feature1 (pts (xy 292.1 156.21) (xy 292.1 179.02142)))
+    (feature2 (pts (xy 215.9 156.21) (xy 215.9 179.02142)))
+    (crossbar (pts (xy 215.9 178.434999) (xy 292.1 178.434999)))
+    (arrow1a (pts (xy 292.1 178.434999) (xy 290.973496 179.02142)))
+    (arrow1b (pts (xy 292.1 178.434999) (xy 290.973496 177.848578)))
+    (arrow2a (pts (xy 215.9 178.434999) (xy 217.026504 179.02142)))
+    (arrow2b (pts (xy 215.9 178.434999) (xy 217.026504 177.848578)))
+  )
+  (dimension 38.1 (width 0.15) (layer Dwgs.User)
+    (gr_text "1.5000 in" (at 196.85 179.735) (layer Dwgs.User)
+      (effects (font (size 1 1) (thickness 0.15)))
+    )
+    (feature1 (pts (xy 215.9 156.21) (xy 215.9 179.021421)))
+    (feature2 (pts (xy 177.8 156.21) (xy 177.8 179.021421)))
+    (crossbar (pts (xy 177.8 178.435) (xy 215.9 178.435)))
+    (arrow1a (pts (xy 215.9 178.435) (xy 214.773496 179.021421)))
+    (arrow1b (pts (xy 215.9 178.435) (xy 214.773496 177.848579)))
+    (arrow2a (pts (xy 177.8 178.435) (xy 178.926504 179.021421)))
+    (arrow2b (pts (xy 177.8 178.435) (xy 178.926504 177.848579)))
+  )
+  (dimension 76.2 (width 0.15) (layer Dwgs.User)
+    (gr_text "3.0000 in" (at 139.7 179.734999) (layer Dwgs.User)
+      (effects (font (size 1 1) (thickness 0.15)))
+    )
+    (feature1 (pts (xy 177.8 156.21) (xy 177.8 179.02142)))
+    (feature2 (pts (xy 101.6 156.21) (xy 101.6 179.02142)))
+    (crossbar (pts (xy 101.6 178.434999) (xy 177.8 178.434999)))
+    (arrow1a (pts (xy 177.8 178.434999) (xy 176.673496 179.02142)))
+    (arrow1b (pts (xy 177.8 178.434999) (xy 176.673496 177.848578)))
+    (arrow2a (pts (xy 101.6 178.434999) (xy 102.726504 179.02142)))
+    (arrow2b (pts (xy 101.6 178.434999) (xy 102.726504 177.848578)))
+  )
+  (dimension 298.45 (width 0.15) (layer Dwgs.User)
+    (gr_text "11.7500 in" (at 196.85 56.485001) (layer Dwgs.User)
+      (effects (font (size 1 1) (thickness 0.15)))
+    )
+    (feature1 (pts (xy 47.625 68.58) (xy 47.625 57.19858)))
+    (feature2 (pts (xy 346.075 68.58) (xy 346.075 57.19858)))
+    (crossbar (pts (xy 346.075 57.785001) (xy 47.625 57.785001)))
+    (arrow1a (pts (xy 47.625 57.785001) (xy 48.751504 57.19858)))
+    (arrow1b (pts (xy 47.625 57.785001) (xy 48.751504 58.371422)))
+    (arrow2a (pts (xy 346.075 57.785001) (xy 344.948496 57.19858)))
+    (arrow2b (pts (xy 346.075 57.785001) (xy 344.948496 58.371422)))
+  )
+  (dimension 292.1 (width 0.15) (layer Dwgs.User)
+    (gr_text "11.5000 in" (at 196.85 60.295) (layer Dwgs.User)
+      (effects (font (size 1 1) (thickness 0.15)))
+    )
+    (feature1 (pts (xy 342.9 68.58) (xy 342.9 61.008579)))
+    (feature2 (pts (xy 50.8 68.58) (xy 50.8 61.008579)))
+    (crossbar (pts (xy 50.8 61.595) (xy 342.9 61.595)))
+    (arrow1a (pts (xy 342.9 61.595) (xy 341.773496 62.181421)))
+    (arrow1b (pts (xy 342.9 61.595) (xy 341.773496 61.008579)))
+    (arrow2a (pts (xy 50.8 61.595) (xy 51.926504 62.181421)))
+    (arrow2b (pts (xy 50.8 61.595) (xy 51.926504 61.008579)))
+  )
   (gr_text SEGMENT-60 (at 196.85 151.765) (layer B.SilkS)
     (effects (font (size 2 2) (thickness 0.3)) (justify mirror))
@@
     (polygon
       (pts
-        (xy 347.98 177.8) (xy 45.72 177.8) (xy 45.72 63.5) (xy 347.98 63.5)
-      )
-    )
-  )
-  (zone (net 90) (net_name GND) (layer B.Cu) (hatch edge 0.508)
-    (priority 1)
-    (connect_pads yes (clearance 0.381))
-    (min_thickness 0.254)
-    (fill yes (arc_segments 32) (thermal_gap 0.508) (thermal_bridge_width 0.508))
-    (polygon
-      (pts
-        (xy 347.98 177.8) (xy 45.72 177.8) (xy 45.72 63.5) (xy 347.98 63.5)
+        (xy 347.98 176.53) (xy 45.72 176.53) (xy 45.72 63.5) (xy 347.98 63.5)
       )
     )
@@
       )
     )
+  )
+  (zone (net 90) (net_name GND) (layer B.Cu) (hatch edge 0.508)
+    (priority 1)
+    (connect_pads yes (clearance 0.381))
+    (min_thickness 0.254)
+    (fill yes (arc_segments 32) (thermal_gap 0.508) (thermal_bridge_width 0.508))
+    (polygon
+      (pts
+        (xy 347.98 176.53) (xy 45.72 176.53) (xy 45.72 63.5) (xy 347.98 63.5)
+      )
+    )
