File: segment_60_PCB/segment_60_PCB.sch (KiCad schematic (older format))
At the start: 122 parts, among them J2 #AVR-ISP-6, SW1 SW_Push, U4 74HC138, Y1 12MHz

Commit message: Updated KiCAD project names in preparation for new keyboards; minor changes to SEGMENT-60 schematic.
Parts:
- removed R?: 10k, Resistor_THT:R_Axial_DIN0204_L3.6mm_D1.6mm_P5.08mm_Horizontal, symbol Device:R
- C?: renamed from C7; value 22p -> 27p
- C?: renamed from C6; value 22p -> 27p
- R? (x2): value 68R -> 75R
- renumbered C4 to C?, C5 to C?, C3 to C?, D3 to D?, J2 to J?, R5 to R?, R6 to R?, SW1 to SW?, U4 to U?, Y1 to Y?
Connections:
- net labels removed: SCL, SDA
- wire segments 476 -> 473
- no-connect marks 23 -> 25
