File: segment_60_PCB/segment_60_PCB.sch (KiCad schematic (older format))
At the start: 123 parts, among them J1 MDB-9M, J2 #AVR-ISP-6, SW1 SW_Push_45deg, SW10 SW_Push_45deg, SW11 SW_Push_45deg, SW12 SW_Push_45deg, SW13 SW_Push_45deg, SW14 SW_Push_45deg, SW15 SW_Push_45deg, SW16 SW_Push_45deg, SW17 SW_Push_45deg, SW18 SW_Push_45deg, SW19 SW_Push_45deg, SW2 SW_Push_45deg, SW20 SW_Push_45deg, SW21 SW_Push_45deg, SW22 SW_Push_45deg, SW23 SW_Push_45deg, SW24 SW_Push_45deg, SW25 SW_Push_45deg, SW26 SW_Push_45deg, SW27 SW_Push_45deg, SW28 SW_Push_45deg, SW29 SW_Push_45deg, SW3 SW_Push_45deg, SW30 SW_Push_45deg, SW31 SW_Push_45deg, SW32 SW_Push_45deg, SW33 SW_Push_45deg, SW34 SW_Push_45deg, SW35 SW_Push_45deg, SW36 SW_Push_45deg, SW37 SW_Push_45deg, SW38 SW_Push_45deg, SW39 SW_Push_45deg, SW4 SW_Push_45deg, SW40 SW_Push_45deg, SW41 SW_Push_45deg, SW42 SW_Push_45deg, SW43 SW_Push_45deg, SW44 SW_Push_45deg, SW45 SW_Push_45deg, SW46 SW_Push_45deg, SW47 SW_Push_45deg, SW48 SW_Push_45deg, SW49 SW_Push_45deg, SW5 SW_Push_45deg, SW50 SW_Push_45deg, SW51 SW_Push_45deg, SW52 SW_Push_45deg, SW53 SW_Push_45deg, SW54 SW_Push_45deg, SW55 SW_Push_45deg, SW56 SW_Push_45deg, SW57 SW_Push_45deg, SW58 SW_Push_45deg, SW59 SW_Push_45deg, SW6 SW_Push_45deg, SW60 SW_Push_45deg, SW61 SW_Push_45deg, SW62 SW_Push_45deg, SW63 SW_Push_45deg, SW64 SW_Push_45deg, SW65 SW_Push_45deg, SW66 SW_Push, SW67 SW_Push, SW7 SW_Push_45deg, SW8 SW_Push_45deg, SW9 SW_Push_45deg, U1 ATmega328P-PU, U10 74HC365, U11 74HC365, U12 74HC365, U13 74HC365, U14 74HC365, U15 74HC365, U16 74HC365, U17 74HC365, U2 74HC138, U3 74HC138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

Commit message: Updated keyswitch footprints to correct sizes.
Parts:
- SW14: footprint Segment_Footprints:Segment_MX_1.00u_PCB -> Segment_Footprints:Segment_MX_1.00u_2.00u_PCB
- SW15, SW57, SW59, SW63, SW65: footprint Segment_Footprints:Segment_MX_1.00u_PCB -> Segment_Footprints:Segment_MX_1.50u_PCB
- SW29: footprint Segment_Footprints:Segment_MX_1.00u_PCB -> Segment_Footprints:Segment_MX_1.25u_1.75u_PCB
- SW41: footprint Segment_Footprints:Segment_MX_1.00u_PCB -> Segment_Footprints:Segment_MX_1.00u_2.25u_PCB
- SW42: footprint Segment_Footprints:Segment_MX_1.00u_PCB -> Segment_Footprints:Segment_MX_1.50u_ISO_PCB
- SW43: footprint Segment_Footprints:Segment_MX_1.00u_PCB -> Segment_Footprints:Segment_MX_1.25u_2.25u_PCB
- SW55: footprint Segment_Footprints:Segment_MX_1.00u_PCB -> Segment_Footprints:Segment_MX_1.75u_2.75u_PCB
- SW60, SW62: footprint Segment_Footprints:Segment_MX_1.00u_PCB -> Segment_Footprints:Segment_MX_2.75u_PCB
- SW61: footprint Segment_Footprints:Segment_MX_1.00u_PCB -> Segment_Footprints:Segment_MX_7.00u_PCB
Changed lines of the file:
@@
 F 0 "SW43" H 1750 3100 50  0000 C CNN
 F 1 "SW_Push_45deg" H 1550 3390 50  0001 C CNN
-F 2 "Segment_Footprints:Segment_MX_1.00u_PCB" H 1550 3200 50  0001 C CNN
+F 2 "Segment_Footprints:Segment_MX_1.25u_2.25u_PCB" H 1550 3200 50  0001 C CNN
 F 3 "~" H 1550 3200 50  0001 C CNN
 	1    1550 3200
@@
 F 0 "SW57" H 1650 3400 50  0000 C CNN
 F 1 "SW_Push_45deg" H 1450 3690 50  0001 C CNN
-F 2 "Segment_Footprints:Segment_MX_1.00u_PCB" H 1450 3500 50  0001 C CNN
+F 2 "Segment_Footprints:Segment_MX_1.50u_PCB" H 1450 3500 50  0001 C CNN
 F 3 "~" H 1450 3500 50  0001 C CNN
 	1    1450 3500
@@
 F 0 "SW29" H 1850 2800 50  0000 C CNN
 F 1 "SW_Push_45deg" H 1650 3090 50  0001 C CNN
-F 2 "Segment_Footprints:Segment_MX_1.00u_PCB" H 1650 2900 50  0001 C CNN
+F 2 "Segment_Footprints:Segment_MX_1.25u_1.75u_PCB" H 1650 2900 50  0001 C CNN
 F 3 "~" H 1650 2900 50  0001 C CNN
 	1    1650 2900
@@
 F 0 "SW15" H 1950 2500 50  0000 C CNN
 F 1 "SW_Push_45deg" H 1750 2790 50  0001 C CNN
-F 2 "Segment_Footprints:Segment_MX_1.00u_PCB" H 1750 2600 50  0001 C CNN
+F 2 "Segment_Footprints:Segment_MX_1.50u_PCB" H 1750 2600 50  0001 C CNN
 F 3 "~" H 1750 2600 50  0001 C CNN
 	1    1750 2600
@@
 F 0 "SW59" H 4950 3400 50  0000 C CNN
 F 1 "SW_Push_45deg" H 4750 3690 50  0001 C CNN
-F 2 "Segment_Footprints:Segment_MX_1.00u_PCB" H 4750 3500 50  0001 C CNN
+F 2 "Segment_Footprints:Segment_MX_1.50u_PCB" H 4750 3500 50  0001 C CNN
 F 3 "~" H 4750 3500 50  0001 C CNN
 	1    4750 3500
@@
 F 0 "SW60" H 9900 3400 50  0000 C CNN
 F 1 "SW_Push_45deg" H 9700 3690 50  0001 C CNN
-F 2 "Segment_Footprints:Segment_MX_1.00u_PCB" H 9700 3500 50  0001 C CNN
+F 2 "Segment_Footprints:Segment_MX_2.75u_PCB" H 9700 3500 50  0001 C CNN
 F 3 "~" H 9700 3500 50  0001 C CNN
 	1    9700 3500
@@
 F 0 "SW61" H 1650 6600 50  0000 C CNN
 F 1 "SW_Push_45deg" H 1450 6890 50  0001 C CNN
-F 2 "Segment_Footprints:Segment_MX_1.00u_PCB" H 1450 6700 50  0001 C CNN
+F 2 "Segment_Footprints:Segment_MX_7.00u_PCB" H 1450 6700 50  0001 C CNN
 F 3 "~" H 1450 6700 50  0001 C CNN
 	1    1450 6700
@@
 F 0 "SW62" H 4950 6600 50  0000 C CNN
 F 1 "SW_Push_45deg" H 4750 6890 50  0001 C CNN
-F 2 "Segment_Footprints:Segment_MX_1.00u_PCB" H 4750 6700 50  0001 C CNN
+F 2 "Segment_Footprints:Segment_MX_2.75u_PCB" H 4750 6700 50  0001 C CNN
 F 3 "~" H 4750 6700 50  0001 C CNN
 	1    4750 6700
@@
 F 0 "SW63" H 8250 6600 50  0000 C CNN
 F 1 "SW_Push_45deg" H 8050 6890 50  0001 C CNN
-F 2 "Segment_Footprints:Segment_MX_1.00u_PCB" H 8050 6700 50  0001 C CNN
+F 2 "Segment_Footprints:Segment_MX_1.50u_PCB" H 8050 6700 50  0001 C CNN
 F 3 "~" H 8050 6700 50  0001 C CNN
 	1    8050 6700
@@
 F 0 "SW55" H 10000 6300 50  0000 C CNN
 F 1 "SW_Push_45deg" H 9800 6590 50  0001 C CNN
-F 2 "Segment_Footprints:Segment_MX_1.00u_PCB" H 9800 6400 50  0001 C CNN
+F 2 "Segment_Footprints:Segment_MX_1.75u_2.75u_PCB" H 9800 6400 50  0001 C CNN
 F 3 "~" H 9800 6400 50  0001 C CNN
 	1    9800 6400
@@
 F 0 "SW41" H 10100 6000 50  0000 C CNN
 F 1 "SW_Push_45deg" H 9900 6290 50  0001 C CNN
-F 2 "Segment_Footprints:Segment_MX_1.00u_PCB" H 9900 6100 50  0001 C CNN
+F 2 "Segment_Footprints:Segment_MX_1.00u_2.25u_PCB" H 9900 6100 50  0001 C CNN
 F 3 "~" H 9900 6100 50  0001 C CNN
 	1    9900 6100
@@
 F 0 "SW65" H 11550 6600 50  0000 C CNN
 F 1 "SW_Push_45deg" H 11350 6890 50  0001 C CNN
-F 2 "Segment_Footprints:Segment_MX_1.00u_PCB" H 11350 6700 50  0001 C CNN
+F 2 "Segment_Footprints:Segment_MX_1.50u_PCB" H 11350 6700 50  0001 C CNN
 F 3 "~" H 11350 6700 50  0001 C CNN
 	1    11350 6700
@@
 F 0 "SW42" H 11750 6000 50  0000 C CNN
 F 1 "SW_Push_45deg" H 11550 6290 50  0001 C CNN
-F 2 "Segment_Footprints:Segment_MX_1.00u_PCB" H 11550 6100 50  0001 C CNN
+F 2 "Segment_Footprints:Segment_MX_1.50u_ISO_PCB" H 11550 6100 50  0001 C CNN
 F 3 "~" H 11550 6100 50  0001 C CNN
 	1    11550 6100
@@
 F 0 "SW14" H 11950 5400 50  0000 C CNN
 F 1 "SW_Push_45deg" H 11750 5690 50  0001 C CNN
-F 2 "Segment_Footprints:Segment_MX_1.00u_PCB" H 11750 5500 50  0001 C CNN
+F 2 "Segment_Footprints:Segment_MX_1.00u_2.00u_PCB" H 11750 5500 50  0001 C CNN
 F 3 "~" H 11750 5500 50  0001 C CNN
 	1    11750 5500

Commit message: Started SEGMENT 60 layout
Parts:
- C10, C11, C12, C13, C14, C15, C16, C17, C18, C19, C20, C5, C6, C7, C8, C9: footprint Capacitor_THT:C_Disc_D3.0mm_W1.6mm_P2.50mm -> Capacitor_THT:C_Axial_L3.8mm_D2.6mm_P7.50mm_Horizontal
- J1: footprint (none) -> Connector_Dsub:DSUB-9_Female_Horizontal_P2.77x2.84mm_EdgePinOffset4.94mm_Housed_MountingHolesOffset7.48mm
- Y1: footprint Crystal:Crystal_HC18-U_Vertical -> Crystal:Crystal_HC49-4H_Vertical
Changed lines of the file:
@@
 F 0 "C6" H 5765 8096 50  0000 L CNN
 F 1 "100n" H 5765 8005 50  0000 L CNN
-F 2 "Capacitor_THT:C_Disc_D3.0mm_W1.6mm_P2.50mm" H 5688 7900 50  0001 C CNN
+F 2 "Capacitor_THT:C_Axial_L3.8mm_D2.6mm_P7.50mm_Horizontal" H 5688 7900 50  0001 C CNN
 F 3 "~" H 5650 8050 50  0001 C CNN
 	1    5650 8050
@@
 F 0 "C5" H 3115 8096 50  0000 L CNN
 F 1 "100n" H 3115 8005 50  0000 L CNN
-F 2 "Capacitor_THT:C_Disc_D3.0mm_W1.6mm_P2.50mm" H 3038 7900 50  0001 C CNN
+F 2 "Capacitor_THT:C_Axial_L3.8mm_D2.6mm_P7.50mm_Horizontal" H 3038 7900 50  0001 C CNN
 F 3 "~" H 3000 8050 50  0001 C CNN
 	1    3000 8050
@@
 F 0 "J1" H 13550 6700 50  0000 C CNN
 F 1 "MDB-9M" H 13550 5550 50  0000 C CNN
-F 2 "" H 13550 6150 50  0001 C CNN
+F 2 "Connector_Dsub:DSUB-9_Female_Horizontal_P2.77x2.84mm_EdgePinOffset4.94mm_Housed_MountingHolesOffset7.48mm" H 13550 6150 50  0001 C CNN
 F 3 " ~" H 13550 6150 50  0001 C CNN
 	1    13550 6150
@@
 F 0 "Y1" H 14300 8718 50  0000 C CNN
 F 1 "16MHz" H 14300 8627 50  0000 C CNN
-F 2 "Crystal:Crystal_HC18-U_Vertical" H 14300 8450 50  0001 C CNN
+F 2 "Crystal:Crystal_HC49-4H_Vertical" H 14300 8450 50  0001 C CNN
 F 3 "~" H 14300 8450 50  0001 C CNN
 	1    14300 8450
@@
 F 0 "C7" H 2215 1846 50  0000 L CNN
 F 1 "100n" H 2215 1755 50  0000 L CNN
-F 2 "Capacitor_THT:C_Disc_D3.0mm_W1.6mm_P2.50mm" H 2138 1650 50  0001 C CNN
+F 2 "Capacitor_THT:C_Axial_L3.8mm_D2.6mm_P7.50mm_Horizontal" H 2138 1650 50  0001 C CNN
 F 3 "~" H 2100 1800 50  0001 C CNN
 	1    2100 1800
@@
 F 0 "C8" H 3865 1846 50  0000 L CNN
 F 1 "100n" H 3865 1755 50  0000 L CNN
-F 2 "Capacitor_THT:C_Disc_D3.0mm_W1.6mm_P2.50mm" H 3788 1650 50  0001 C CNN
+F 2 "Capacitor_THT:C_Axial_L3.8mm_D2.6mm_P7.50mm_Horizontal" H 3788 1650 50  0001 C CNN
 F 3 "~" H 3750 1800 50  0001 C CNN
 	1    3750 1800
@@
 F 0 "C9" H 5515 1846 50  0000 L CNN
 F 1 "100n" H 5515 1755 50  0000 L CNN
-F 2 "Capacitor_THT:C_Disc_D3.0mm_W1.6mm_P2.50mm" H 5438 1650 50  0001 C CNN
+F 2 "Capacitor_THT:C_Axial_L3.8mm_D2.6mm_P7.50mm_Horizontal" H 5438 1650 50  0001 C CNN
 F 3 "~" H 5400 1800 50  0001 C CNN
 	1    5400 1800
@@
 F 0 "C10" H 7165 1846 50  0000 L CNN
 F 1 "100n" H 7165 1755 50  0000 L CNN
-F 2 "Capacitor_THT:C_Disc_D3.0mm_W1.6mm_P2.50mm" H 7088 1650 50  0001 C CNN
+F 2 "Capacitor_THT:C_Axial_L3.8mm_D2.6mm_P7.50mm_Horizontal" H 7088 1650 50  0001 C CNN
 F 3 "~" H 7050 1800 50  0001 C CNN
 	1    7050 1800
@@
 F 0 "C11" H 8815 1846 50  0000 L CNN
 F 1 "100n" H 8815 1755 50  0000 L CNN
-F 2 "Capacitor_THT:C_Disc_D3.0mm_W1.6mm_P2.50mm" H 8738 1650 50  0001 C CNN
+F 2 "Capacitor_THT:C_Axial_L3.8mm_D2.6mm_P7.50mm_Horizontal" H 8738 1650 50  0001 C CNN
 F 3 "~" H 8700 1800 50  0001 C CNN
 	1    8700 1800
@@
 F 0 "C12" H 10465 1846 50  0000 L CNN
 F 1 "100n" H 10465 1755 50  0000 L CNN
-F 2 "Capacitor_THT:C_Disc_D3.0mm_W1.6mm_P2.50mm" H 10388 1650 50  0001 C CNN
+F 2 "Capacitor_THT:C_Axial_L3.8mm_D2.6mm_P7.50mm_Horizontal" H 10388 1650 50  0001 C CNN
 F 3 "~" H 10350 1800 50  0001 C CNN
 	1    10350 1800
@@
 F 0 "C13" H 12115 1846 50  0000 L CNN
 F 1 "100n" H 12115 1755 50  0000 L CNN
-F 2 "Capacitor_THT:C_Disc_D3.0mm_W1.6mm_P2.50mm" H 12038 1650 50  0001 C CNN
+F 2 "Capacitor_THT:C_Axial_L3.8mm_D2.6mm_P7.50mm_Horizontal" H 12038 1650 50  0001 C CNN
 F 3 "~" H 12000 1800 50  0001 C CNN
 	1    12000 1800
@@
 F 0 "C14" H 2215 5046 50  0000 L CNN
 F 1 "100n" H 2215 4955 50  0000 L CNN
-F 2 "Capacitor_THT:C_Disc_D3.0mm_W1.6mm_P2.50mm" H 2138 4850 50  0001 C CNN
+F 2 "Capacitor_THT:C_Axial_L3.8mm_D2.6mm_P7.50mm_Horizontal" H 2138 4850 50  0001 C CNN
 F 3 "~" H 2100 5000 50  0001 C CNN
 	1    2100 5000
@@
 F 0 "C15" H 3865 5046 50  0000 L CNN
 F 1 "100n" H 3865 4955 50  0000 L CNN
-F 2 "Capacitor_THT:C_Disc_D3.0mm_W1.6mm_P2.50mm" H 3788 4850 50  0001 C CNN
+F 2 "Capacitor_THT:C_Axial_L3.8mm_D2.6mm_P7.50mm_Horizontal" H 3788 4850 50  0001 C CNN
 F 3 "~" H 3750 5000 50  0001 C CNN
 	1    3750 5000
@@
 F 0 "C16" H 5515 5046 50  0000 L CNN
 F 1 "100n" H 5515 4955 50  0000 L CNN
-F 2 "Capacitor_THT:C_Disc_D3.0mm_W1.6mm_P2.50mm" H 5438 4850 50  0001 C CNN
+F 2 "Capacitor_THT:C_Axial_L3.8mm_D2.6mm_P7.50mm_Horizontal" H 5438 4850 50  0001 C CNN
 F 3 "~" H 5400 5000 50  0001 C CNN
 	1    5400 5000
@@
 F 0 "C17" H 7165 5046 50  0000 L CNN
 F 1 "100n" H 7165 4955 50  0000 L CNN
-F 2 "Capacitor_THT:C_Disc_D3.0mm_W1.6mm_P2.50mm" H 7088 4850 50  0001 C CNN
+F 2 "Capacitor_THT:C_Axial_L3.8mm_D2.6mm_P7.50mm_Horizontal" H 7088 4850 50  0001 C CNN
 F 3 "~" H 7050 5000 50  0001 C CNN
 	1    7050 5000
@@
 F 0 "C18" H 8815 5046 50  0000 L CNN
 F 1 "100n" H 8815 4955 50  0000 L CNN
-F 2 "Capacitor_THT:C_Disc_D3.0mm_W1.6mm_P2.50mm" H 8738 4850 50  0001 C CNN
+F 2 "Capacitor_THT:C_Axial_L3.8mm_D2.6mm_P7.50mm_Horizontal" H 8738 4850 50  0001 C CNN
 F 3 "~" H 8700 5000 50  0001 C CNN
 	1    8700 5000
@@
 F 0 "C19" H 10465 5046 50  0000 L CNN
 F 1 "100n" H 10465 4955 50  0000 L CNN
-F 2 "Capacitor_THT:C_Disc_D3.0mm_W1.6mm_P2.50mm" H 10388 4850 50  0001 C CNN
+F 2 "Capacitor_THT:C_Axial_L3.8mm_D2.6mm_P7.50mm_Horizontal" H 10388 4850 50  0001 C CNN
 F 3 "~" H 10350 5000 50  0001 C CNN
 	1    10350 5000
@@
 F 0 "C20" H 12115 5046 50  0000 L CNN
 F 1 "100n" H 12115 4955 50  0000 L CNN
-F 2 "Capacitor_THT:C_Disc_D3.0mm_W1.6mm_P2.50mm" H 12038 4850 50  0001 C CNN
+F 2 "Capacitor_THT:C_Axial_L3.8mm_D2.6mm_P7.50mm_Horizontal" H 12038 4850 50  0001 C CNN
 F 3 "~" H 12000 5000 50  0001 C CNN
 	1    12000 5000

Commit message: Continued organizing footprints and minor layout changes to control hardware.
Parts:
- C1: footprint Capacitor_THT:C_Disc_D3.0mm_W1.6mm_P2.50mm -> Capacitor_THT:C_Axial_L3.8mm_D2.6mm_P7.50mm_Horizontal
- D1, D2: footprint Diode_THT:D_DO-35_SOD27_P7.62mm_Horizontal -> Diode_THT:D_DO-35_SOD27_P10.16mm_Horizontal
Changed lines of the file:
@@
 F 0 "C1" H 15300 1300 50  0000 L CNN
 F 1 "100n" H 15300 1100 50  0000 L CNN
-F 2 "Capacitor_THT:C_Disc_D3.0mm_W1.6mm_P2.50mm" H 15288 1050 50  0001 C CNN
+F 2 "Capacitor_THT:C_Axial_L3.8mm_D2.6mm_P7.50mm_Horizontal" H 15288 1050 50  0001 C CNN
 F 3 "~" H 15250 1200 50  0001 C CNN
 	1    15250 1200
@@
 F 0 "D1" V 14350 6525 50  0000 L CNN
 F 1 "3.6V" V 14550 6525 50  0000 L CNN
-F 2 "Diode_THT:D_DO-35_SOD27_P7.62mm_Horizontal" H 14450 6500 50  0001 C CNN
+F 2 "Diode_THT:D_DO-35_SOD27_P10.16mm_Horizontal" H 14450 6500 50  0001 C CNN
 F 3 "~" H 14450 6500 50  0001 C CNN
 	1    14450 6500
@@
 F 0 "D2" V 14600 6525 50  0000 L CNN
 F 1 "3.6V" V 14800 6525 50  0000 L CNN
-F 2 "Diode_THT:D_DO-35_SOD27_P7.62mm_Horizontal" H 14700 6500 50  0001 C CNN
+F 2 "Diode_THT:D_DO-35_SOD27_P10.16mm_Horizontal" H 14700 6500 50  0001 C CNN
 F 3 "~" H 14700 6500 50  0001 C CNN
 	1    14700 6500

Commit message: Added remaining footprints, changed library paths to be relative.
Parts:
- C1: footprint Capacitor_THT:C_Axial_L3.8mm_D2.6mm_P7.50mm_Horizontal -> Capacitor_THT:C_Axial_L3.8mm_D2.6mm_P10.00mm_Horizontal
- C4: footprint (none) -> Capacitor_THT:CP_Axial_L11.0mm_D5.0mm_P18.00mm_Horizontal
- F1: footprint (none) -> Fuse:Fuse_Littelfuse_395Series
- SW66, SW67: footprint (none) -> Button_Switch_THT:SW_PUSH_6mm
Connections:
- wire segments 597 -> 595
Other:
- moved on the sheet: C4, D1, D2, F1, R1, R2, R3
Changed lines of the file:
@@
 F 0 "SW66" V 8946 8602 50  0000 R CNN
 F 1 "SW_Push" V 8855 8602 50  0000 R CNN
-F 2 "" H 8900 8850 50  0001 C CNN
+F 2 "Button_Switch_THT:SW_PUSH_6mm" H 8900 8850 50  0001 C CNN
 F 3 "~" H 8900 8850 50  0001 C CNN
 	1    8900 8650
@@
 	1    0    0    -1
 $EndComp
-Text GLabel 15050 6250 2    50   Input ~ 0
+Text GLabel 15000 6250 2    50   Input ~ 0
 D+
-Text GLabel 15050 6050 2    50   Input ~ 0
+Text GLabel 15000 6050 2    50   Input ~ 0
 D-
 $Comp
 L Device:R R3
 U 1 1 5FC489A0
-P 14900 6250
-F 0 "R3" V 14975 6350 50  0000 C CNN
-F 1 "75R" V 14975 6175 50  0000 C CNN
-F 2 "Resistor_THT:R_Axial_DIN0207_L6.3mm_D2.5mm_P10.16mm_Horizontal" V 14830 6250 50  0001 C CNN
-F 3 "~" H 14900 6250 50  0001 C CNN
-	1    14900 6250
+P 14850 6250
+F 0 "R3" V 14925 6350 50  0000 C CNN
+F 1 "75R" V 14925 6175 50  0000 C CNN
+F 2 "Resistor_THT:R_Axial_DIN0207_L6.3mm_D2.5mm_P10.16mm_Horizontal" V 14780 6250 50  0001 C CNN
+F 3 "~" H 14850 6250 50  0001 C CNN
+	1    14850 6250
 	0    -1   -1   0
 $EndComp
@@
 L Device:R R2
 U 1 1 5FC489B2
-P 14900 6050
-F 0 "R2" V 14975 6150 50  0000 C CNN
-F 1 "75R" V 14975 5975 50  0000 C CNN
-F 2 "Resistor_THT:R_Axial_DIN0207_L6.3mm_D2.5mm_P10.16mm_Horizontal" V 14830 6050 50  0001 C CNN
-F 3 "~" H 14900 6050 50  0001 C CNN
-	1    14900 6050
+P 14850 6050
+F 0 "R2" V 14925 6150 50  0000 C CNN
+F 1 "75R" V 14925 5975 50  0000 C CNN
+F 2 "Resistor_THT:R_Axial_DIN0207_L6.3mm_D2.5mm_P10.16mm_Horizontal" V 14780 6050 50  0001 C CNN
+F 3 "~" H 14850 6050 50  0001 C CNN
+	1    14850 6050
 	0    -1   -1   0
 $EndComp
@@
 L power:VCC #PWR07
 U 1 1 5FC489D2
-P 14100 5250
-F 0 "#PWR07" H 14100 5100 50  0001 C CNN
-F 1 "VCC" H 14115 5423 50  0000 C CNN
-F 2 "" H 14100 5250 50  0001 C CNN
-F 3 "" H 14100 5250 50  0001 C CNN
-	1    14100 5250
+P 14150 5250
+F 0 "#PWR07" H 14150 5100 50  0001 C CNN
+F 1 "VCC" H 14165 5423 50  0000 C CNN
+F 2 "" H 14150 5250 50  0001 C CNN
+F 3 "" H 14150 5250 50  0001 C CNN
+	1    14150 5250
 	1    0    0    -1
 $EndComp
@@
 L Device:Polyfuse F1
 U 1 1 5FC489D8
-P 14100 5500
-F 0 "F1" H 14188 5546 50  0000 L CNN
-F 1 "100mA" H 14188 5455 50  0000 L CNN
-F 2 "" H 14150 5300 50  0001 L CNN
-F 3 "~" H 14100 5500 50  0001 C CNN
-	1    14100 5500
+P 14150 5500
+F 0 "F1" H 14238 5546 50  0000 L CNN
+F 1 "100mA" H 14238 5455 50  0000 L CNN
+F 2 "Fuse:Fuse_Littelfuse_395Series" H 14200 5300 50  0001 L CNN
+F 3 "~" H 14150 5500 50  0001 C CNN
+	1    14150 5500
 	-1   0    0    -1
 $EndComp
@@
 L Device:R R1
 U 1 1 5FC489EA
-P 14450 5500
-F 0 "R1" H 14520 5546 50  0000 L CNN
-F 1 "1.5k" H 14520 5455 50  0000 L CNN
-F 2 "Resistor_THT:R_Axial_DIN0207_L6.3mm_D2.5mm_P10.16mm_Horizontal" V 14380 5500 50  0001 C CNN
-F 3 "~" H 14450 5500 50  0001 C CNN
-	1    14450 5500
+P 14400 5500
+F 0 "R1" H 14470 5546 50  0000 L CNN
+F 1 "1.5k" H 14470 5455 50  0000 L CNN
+F 2 "Resistor_THT:R_Axial_DIN0207_L6.3mm_D2.5mm_P10.16mm_Horizontal" V 14330 5500 50  0001 C CNN
+F 3 "~" H 14400 5500 50  0001 C CNN
+	1    14400 5500
 	1    0    0    -1
 $EndComp
-$Comp
-L power:GND #PWR08
-U 1 1 5FC489F0
-P 14900 5650
-F 0 "#PWR08" H 14900 5400 50  0001 C CNN
-F 1 "GND" H 14905 5477 50  0000 C CNN
-F 2 "" H 14900 5650 50  0001 C CNN
-F 3 "" H 14900 5650 50  0001 C CNN
-	1    14900 5650
-	1    0    0    -1
-$EndComp
-$Comp
-L Device:C C4
-U 1 1 5FC489F6
-P 14900 5500
-F 0 "C4" H 15015 5546 50  0000 L CNN
-F 1 "4.7u" H 15015 5455 50  0000 L CNN
-F 2 "" H 14938 5350 50  0001 C CNN
-F 3 "~" H 14900 5500 50  0001 C CNN
-	1    14900 5500
-	1    0    0    -1
-$EndComp
-Wire Wire Line
-	14900 5350 14900 5300
-Wire Wire Line
-	14900 5300 14450 5300
 Wire Wire Line
-	14450 5350 14450 5300
-Connection ~ 14450 5300
+	14400 5350 14400 5300
 $Comp
 L power:GND #PWR03
@@
 F 0 "C1" H 15300 1300 50  0000 L CNN
 F 1 "100n" H 15300 1100 50  0000 L CNN
-F 2 "Capacitor_THT:C_Axial_L3.8mm_D2.6mm_P7.50mm_Horizontal" H 15288 1050 50  0001 C CNN
+F 2 "Capacitor_THT:C_Axial_L3.8mm_D2.6mm_P10.00mm_Horizontal" H 15288 1050 50  0001 C CNN
 F 3 "~" H 15250 1200 50  0001 C CNN
 	1    15250 1200
@@
 $EndComp
 Wire Wire Line
-	14450 6050 14450 5650
+	14400 6050 14400 5650
 $Comp
 L Device:D_Zener D1
 U 1 1 5FC489C0
-P 14450 6500
-F 0 "D1" V 14350 6525 50  0000 L CNN
-F 1 "3.6V" V 14550 6525 50  0000 L CNN
-F 2 "Diode_THT:D_DO-35_SOD27_P10.16mm_Horizontal" H 14450 6500 50  0001 C CNN
-F 3 "~" H 14450 6500 50  0001 C CNN
-	1    14450 6500
+P 14400 6500
+F 0 "D1" V 14300 6525 50  0000 L CNN
+F 1 "3.6V" V 14500 6525 50  0000 L CNN
+F 2 "Diode_THT:D_DO-35_SOD27_P10.16mm_Horizontal" H 14400 6500 50  0001 C CNN
+F 3 "~" H 14400 6500 50  0001 C CNN
+	1    14400 6500
 	0    1    1    0
 $EndComp
@@
 L Device:D_Zener D2
 U 1 1 5FC489BA
-P 14700 6500
-F 0 "D2" V 14600 6525 50  0000 L CNN
-F 1 "3.6V" V 14800 6525 50  0000 L CNN
-F 2 "Diode_THT:D_DO-35_SOD27_P10.16mm_Horizontal" H 14700 6500 50  0001 C CNN
-F 3 "~" H 14700 6500 50  0001 C CNN
-	1    14700 6500
+P 14650 6500
+F 0 "D2" V 14550 6525 50  0000 L CNN
+F 1 "3.6V" V 14750 6525 50  0000 L CNN
+F 2 "Diode_THT:D_DO-35_SOD27_P10.16mm_Horizontal" H 14650 6500 50  0001 C CNN
+F 3 "~" H 14650 6500 50  0001 C CNN
+	1    14650 6500
 	0    1    1    0
 $EndComp
@@
 L power:GND #PWR010
 U 1 1 5FC489AC
-P 14450 6650
-F 0 "#PWR010" H 14450 6400 50  0001 C CNN
-F 1 "GND" H 14455 6477 50  0000 C CNN
-F 2 "" H 14450 6650 50  0001 C CNN
-F 3 "" H 14450 6650 50  0001 C CNN
-	1    14450 6650
+P 14400 6650
+F 0 "#PWR010" H 14400 6400 50  0001 C CNN
+F 1 "GND" H 14405 6477 50  0000 C CNN
+F 2 "" H 14400 6650 50  0001 C CNN
+F 3 "" H 14400 6650 50  0001 C CNN
+	1    14400 6650
 	1    0    0    -1
 $EndComp
@@
 L power:GND #PWR011
 U 1 1 5FC489A6
-P 14700 6650
-F 0 "#PWR011" H 14700 6400 50  0001 C CNN
-F 1 "GND" H 14705 6477 50  0000 C CNN
-F 2 "" H 14700 6650 50  0001 C CNN
-F 3 "" H 14700 6650 50  0001 C CNN
-	1    14700 6650
+P 14650 6650
+F 0 "#PWR011" H 14650 6400 50  0001 C CNN
+F 1 "GND" H 14655 6477 50  0000 C CNN
+F 2 "" H 14650 6650 50  0001 C CNN
+F 3 "" H 14650 6650 50  0001 C CNN
+	1    14650 6650
 	1    0    0    -1
 $EndComp
@@
 L power:GND #PWR09
 U 1 1 5FC0DDEF
-P 14200 6650
-F 0 "#PWR09" H 14200 6400 50  0001 C CNN
-F 1 "GND" H 14205 6477 50  0000 C CNN
-F 2 "" H 14200 6650 50  0001 C CNN
-F 3 "" H 14200 6650 50  0001 C CNN
-	1    14200 6650
+P 14150 6650
+F 0 "#PWR09" H 14150 6400 50  0001 C CNN
+F 1 "GND" H 14155 6477 50  0000 C CNN
+F 2 "" H 14150 6650 50  0001 C CNN
+F 3 "" H 14150 6650 50  0001 C CNN
+	1    14150 6650
 	1    0    0    -1
 $EndComp
-Wire Wire Line
-	14450 6050 14700 6050
-Wire Wire Line
-	14750 6050 14700 6050
-Connection ~ 14700 6050
-Wire Wire Line
-	14700 6350 14700 6050
-Wire Wire Line
-	14750 6250 14450 6250
-Wire Wire Line
-	14450 6350 14450 6250
 $Comp
 L Segment_Symbols:74HC138 U2
@@
 F 0 "SW67" V 9696 8602 50  0000 R CNN
 F 1 "SW_Push" V 9605 8602 50  0000 R CNN
-F 2 "" H 9650 8850 50  0001 C CNN
+F 2 "Button_Switch_THT:SW_PUSH_6mm" H 9650 8850 50  0001 C CNN
 F 3 "~" H 9650 8850 50  0001 C CNN
 	1    9650 8650
@@
 Text GLabel 14800 1550 2    50   Input ~ 0
 LED0
-Wire Wire Line
-	13850 6150 14100 6150
-Text GLabel 13850 5750 2    50   Input ~ 0
-RST
 Text GLabel 13850 5950 2    50   Input ~ 0
+RST
+Text GLabel 13850 6150 2    50   Input ~ 0
 SCK
 Text GLabel 13850 6350 2    50   Input ~ 0
@@
 Wire Wire Line
 	1650 8700 1700 8700
-Wire Wire Line
-	14200 5850 14200 6450
-Wire Wire Line
-	14100 5250 14100 5300
-Wire Wire Line
-	14100 5300 14450 5300
-Connection ~ 14100 5300
-Wire Wire Line
-	14100 5300 14100 5350
-Wire Wire Line
-	14100 5650 14100 6150
-Wire Wire Line
-	13850 5850 14200 5850
-Wire Wire Line
-	13850 6450 14200 6450
-Connection ~ 14200 6450
-Wire Wire Line
-	14200 6450 14200 6650
-Wire Wire Line
-	13850 6250 14450 6250
-Connection ~ 14450 6250
-Wire Wire Line
-	13850 6050 14450 6050
-Connection ~ 14450 6050
 Text Label 14800 3450 0    50   ~ 0
 SEL0
@@
 NoConn ~ 5150 8800
 NoConn ~ 5150 8700
+Text GLabel 13850 5750 2    50   Input ~ 0
+BOOT
+Wire Wire Line
+	13850 5850 14150 5850
+Wire Wire Line
+	13850 6450 14150 6450
+Wire Wire Line
+	14150 6450 14150 6650
+Wire Wire Line
+	14150 5650 14150 5850
+Wire Wire Line
+	14150 5250 14150 5300
+Wire Wire Line
+	13850 6050 14400 6050
+Connection ~ 14400 6050
+Wire Wire Line
+	14400 6250 13850 6250
+Wire Wire Line
+	14700 6250 14400 6250
+Connection ~ 14400 6250
+Wire Wire Line
+	14400 6350 14400 6250
+Wire Wire Line
+	14700 6050 14650 6050
+Wire Wire Line
+	14400 6050 14650 6050
+Connection ~ 14650 6050
+Wire Wire Line
+	14650 6350 14650 6050
+Wire Wire Line
+	14400 5300 14150 5300
+Connection ~ 14150 5300
+Wire Wire Line
+	14150 5300 14150 5350
+Connection ~ 14400 5300
+Wire Wire Line
+	14850 5300 14400 5300
+Wire Wire Line
+	14850 5350 14850 5300
+$Comp
+L Device:C C4
+U 1 1 5FC489F6
+P 14850 5500
+F 0 "C4" H 14965 5546 50  0000 L CNN
+F 1 "4.7u" H 14965 5455 50  0000 L CNN
+F 2 "Capacitor_THT:CP_Axial_L11.0mm_D5.0mm_P18.00mm_Horizontal" H 14888 5350 50  0001 C CNN
+F 3 "~" H 14850 5500 50  0001 C CNN
+	1    14850 5500
+	1    0    0    -1
+$EndComp
+$Comp
+L power:GND #PWR08
+U 1 1 5FC489F0
+P 14850 5650
+F 0 "#PWR08" H 14850 5400 50  0001 C CNN
+F 1 "GND" H 14855 5477 50  0000 C CNN
+F 2 "" H 14850 5650 50  0001 C CNN
+F 3 "" H 14850 5650 50  0001 C CNN
+	1    14850 5650
+	1    0    0    -1
+$EndComp
 Wire Bus Line
 	15100 3550 15100 3950

Commit message: Updated layout; changed row pullup resistors to a single resistor network
Parts:
- removed J1: MDB-9M, Connector_Dsub:DSUB-9_Female_Horizontal_P2.77x2.84mm_EdgePinOffset4.94mm_Housed_MountingHolesOffset7.48mm, symbol Connector:DB9_Male
- removed J2: #AVR-ISP-6, Connector_PinHeader_2.54mm:PinHeader_2x03_P2.54mm_Vertical, symbol Connector:AVR-ISP-6
- removed R10, R11, R7, R8, R9: 10k, Resistor_THT:R_Axial_DIN0207_L6.3mm_D2.5mm_P10.16mm_Horizontal, symbol Device:R
- added J1: BREAKOUT, Connector_PinHeader_2.54mm:PinHeader_2x06_P2.54mm_Vertical, symbol Connector_Generic:Conn_02x06_Odd_Even
- added RN1: 10k, Resistor_THT:R_Array_SIP7, symbol Device:R_Network06
Connections:
- net labels added: ROW5, RXD, SEL4, TXD, USB+, USB-
- wire segments 595 -> 591
- no-connect marks 25 -> 22
Other:
- moved on the sheet: C1, C2, C3, U1, Y1
