File: segment_60_PCB/segment_60_PCB.kicad_pcb (KiCad board)
At the start: 2 copper layers, 285.8 x 133.4 mm, 131 parts, among them J1 BREAKOUT, SW1 SW_Push_45deg, SW10 SW_Push_45deg, SW11 SW_Push_45deg, SW12 SW_Push_45deg, SW13 SW_Push_45deg, SW14 SW_Push_45deg, SW15 SW_Push_45deg, SW16 SW_Push_45deg, SW17 SW_Push_45deg, SW18 SW_Push_45deg, SW19 SW_Push_45deg, SW2 SW_Push_45deg, SW20 SW_Push_45deg, SW21 SW_Push_45deg, SW22 SW_Push_45deg, SW23 SW_Push_45deg, SW24 SW_Push_45deg, SW25 SW_Push_45deg, SW26 SW_Push_45deg, SW27 SW_Push_45deg, SW28 SW_Push_45deg, SW29 SW_Push_45deg, SW3 SW_Push_45deg, SW30 SW_Push_45deg, SW31 SW_Push_45deg, SW32 SW_Push_45deg, SW33 SW_Push_45deg, SW34 SW_Push_45deg, SW35 SW_Push_45deg, SW36 SW_Push_45deg, SW37 SW_Push_45deg, SW38 SW_Push_45deg, SW39 SW_Push_45deg, SW4 SW_Push_45deg, SW40 SW_Push_45deg, SW41 SW_Push_45deg, SW42 SW_Push_45deg, SW43 SW_Push_45deg, SW44 SW_Push_45deg, SW45 SW_Push_45deg, SW46 SW_Push_45deg, SW47 SW_Push_45deg, SW48 SW_Push_45deg, SW49 SW_Push_45deg, SW5 SW_Push_45deg, SW50 SW_Push_45deg, SW51 SW_Push_45deg, SW52 SW_Push_45deg, SW53 SW_Push_45deg, SW54 SW_Push_45deg, SW55 SW_Push_45deg, SW56 SW_Push_45deg, SW57 SW_Push_45deg, SW58 SW_Push_45deg, SW59 SW_Push_45deg, SW6 SW_Push_45deg, SW60 SW_Push_45deg, SW61 SW_Push_45deg, SW62 SW_Push_45deg, SW63 SW_Push_45deg, SW64 SW_Push_45deg, SW65 SW_Push_45deg, SW66 SW_Push, SW67 SW_Push, SW7 SW_Push_45deg, SW8 SW_Push_45deg, SW9 SW_Push_45deg, U1 ATmega328P-PU, U10 74HC365, U11 74HC365, U12 74HC365, U13 74HC365, U14 74HC365, U15 74HC365, U16 74HC365, U17 74HC365, U2 74HC138, U3 74HC138, U4 74HC365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

Commit message: Routed first 8 columns of switches
Parts:
- removed H5, H6, H7, H8: MATRIX, MountingHole:MountingHole_3.2mm_M3_Pad
- moved H11 222.1 mm to (102.2, 212.7)
- moved H9 76.2 mm to (200.0, 212.7)
Connections:
- U10 pad 11: Net-(SW49-Pad1) -> Net-(SW7-Pad1)
- U10 pad 13: Net-(U10-Pad13) -> Net-(SW21-Pad1)
- U10 pad 3: Net-(U10-Pad3) -> Net-(SW35-Pad1)
- U10 pad 5: Net-(SW7-Pad1) -> Net-(SW49-Pad1)
- U10 pad 7: Net-(SW21-Pad1) -> Net-(U10-Pad7)
- U10 pad 9: Net-(SW35-Pad1) -> Net-(U10-Pad9)
- U11 pad 11: Net-(SW50-Pad1) -> Net-(SW8-Pad1)
- U11 pad 13: Net-(SW61-Pad1) -> Net-(SW22-Pad1)
- U11 pad 3: Net-(U11-Pad3) -> Net-(SW36-Pad1)
- U11 pad 5: Net-(SW8-Pad1) -> Net-(SW50-Pad1)
- U11 pad 7: Net-(SW22-Pad1) -> Net-(SW61-Pad1)
- U11 pad 9: Net-(SW36-Pad1) -> Net-(U11-Pad9)
- U12 pad 11: Net-(SW51-Pad1) -> Net-(SW9-Pad1)
- U12 pad 13: Net-(U12-Pad13) -> Net-(SW23-Pad1)
- U12 pad 3: Net-(U12-Pad3) -> Net-(SW37-Pad1)
- U12 pad 5: Net-(SW9-Pad1) -> Net-(SW51-Pad1)
- U12 pad 7: Net-(SW23-Pad1) -> Net-(U12-Pad7)
- U12 pad 9: Net-(SW37-Pad1) -> Net-(U12-Pad9)
- U13 pad 11: Net-(SW52-Pad1) -> Net-(SW10-Pad1)
- U13 pad 13: Net-(SW62-Pad1) -> Net-(SW24-Pad1)
- U13 pad 3: Net-(U13-Pad3) -> Net-(SW38-Pad1)
- U13 pad 5: Net-(SW10-Pad1) -> Net-(SW52-Pad1)
- U13 pad 7: Net-(SW24-Pad1) -> Net-(SW62-Pad1)
- U13 pad 9: Net-(SW38-Pad1) -> Net-(U13-Pad9)
- U14 pad 11: Net-(SW53-Pad1) -> Net-(SW11-Pad1)
- U14 pad 13: Net-(U14-Pad13) -> Net-(SW25-Pad1)
- U14 pad 3: Net-(U14-Pad3) -> Net-(SW39-Pad1)
- U14 pad 5: Net-(SW11-Pad1) -> Net-(SW53-Pad1)
- U14 pad 7: Net-(SW25-Pad1) -> Net-(U14-Pad7)
- U14 pad 9: Net-(SW39-Pad1) -> Net-(U14-Pad9)
- U15 pad 11: Net-(SW54-Pad1) -> Net-(SW12-Pad1)
- U15 pad 13: Net-(SW63-Pad1) -> Net-(SW26-Pad1)
- U15 pad 3: Net-(U15-Pad3) -> Net-(SW40-Pad1)
- U15 pad 5: Net-(SW12-Pad1) -> Net-(SW54-Pad1)
- U15 pad 7: Net-(SW26-Pad1) -> Net-(SW63-Pad1)
- U15 pad 9: Net-(SW40-Pad1) -> Net-(U15-Pad9)
- U16 pad 11: Net-(SW55-Pad1) -> Net-(SW13-Pad1)
- U16 pad 13: Net-(SW64-Pad1) -> Net-(SW27-Pad1)
- U16 pad 3: Net-(U16-Pad3) -> Net-(SW41-Pad1)
- U16 pad 5: Net-(SW13-Pad1) -> Net-(SW55-Pad1)
- U16 pad 7: Net-(SW27-Pad1) -> Net-(SW64-Pad1)
- U16 pad 9: Net-(SW41-Pad1) -> Net-(U16-Pad9)
- U17 pad 11: Net-(SW56-Pad1) -> Net-(SW14-Pad1)
- U17 pad 13: Net-(SW65-Pad1) -> Net-(SW28-Pad1)
- U17 pad 3: Net-(U17-Pad3) -> Net-(SW42-Pad1)
- U17 pad 5: Net-(SW14-Pad1) -> Net-(SW56-Pad1)
- U17 pad 7: Net-(SW28-Pad1) -> Net-(SW65-Pad1)
- U17 pad 9: Net-(SW42-Pad1) -> Net-(U17-Pad9)
- U4 pad 11: Net-(SW43-Pad1) -> Net-(SW1-Pad1)
- U4 pad 13: Net-(SW57-Pad1) -> Net-(SW15-Pad1)
- U4 pad 3: Net-(U4-Pad3) -> Net-(SW29-Pad1)
- U4 pad 5: Net-(SW1-Pad1) -> Net-(SW43-Pad1)
- U4 pad 7: Net-(SW15-Pad1) -> Net-(SW57-Pad1)
- U4 pad 9: Net-(SW29-Pad1) -> Net-(U4-Pad9)
- U5 pad 11: Net-(SW44-Pad1) -> Net-(SW2-Pad1)
- U5 pad 13: Net-(SW58-Pad1) -> Net-(SW16-Pad1)
- U5 pad 3: Net-(U5-Pad3) -> Net-(SW30-Pad1)
- U5 pad 5: Net-(SW2-Pad1) -> Net-(SW44-Pad1)
- U5 pad 7: Net-(SW16-Pad1) -> Net-(SW58-Pad1)
- U5 pad 9: Net-(SW30-Pad1) -> Net-(U5-Pad9)
- U6 pad 11: Net-(SW45-Pad1) -> Net-(SW3-Pad1)
- U6 pad 13: Net-(SW59-Pad1) -> Net-(SW17-Pad1)
- U6 pad 3: Net-(U6-Pad3) -> Net-(SW31-Pad1)
- U6 pad 5: Net-(SW3-Pad1) -> Net-(SW45-Pad1)
- U6 pad 7: Net-(SW17-Pad1) -> Net-(U6-Pad7)
- U6 pad 9: Net-(SW31-Pad1) -> Net-(U6-Pad9)
- U7 pad 11: Net-(SW46-Pad1) -> Net-(SW4-Pad1)
- U7 pad 13: Net-(U7-Pad13) -> Net-(SW18-Pad1)
- U7 pad 3: Net-(U7-Pad3) -> Net-(SW32-Pad1)
- U7 pad 5: Net-(SW4-Pad1) -> Net-(SW46-Pad1)
- U7 pad 7: Net-(SW18-Pad1) -> Net-(SW59-Pad1)
- U7 pad 9: Net-(SW32-Pad1) -> Net-(U7-Pad9)
- U8 pad 11: Net-(SW47-Pad1) -> Net-(SW5-Pad1)
- U8 pad 13: Net-(U8-Pad13) -> Net-(SW19-Pad1)
- U8 pad 3: Net-(U8-Pad3) -> Net-(SW33-Pad1)
- U8 pad 5: Net-(SW5-Pad1) -> Net-(SW47-Pad1)
- U8 pad 7: Net-(SW19-Pad1) -> Net-(U8-Pad7)
- U8 pad 9: Net-(SW33-Pad1) -> Net-(U8-Pad9)
- U9 pad 11: Net-(SW48-Pad1) -> Net-(SW6-Pad1)
- U9 pad 13: Net-(SW60-Pad1) -> Net-(SW20-Pad1)
- U9 pad 3: Net-(U9-Pad3) -> Net-(SW34-Pad1)
- U9 pad 5: Net-(SW6-Pad1) -> Net-(SW48-Pad1)
- U9 pad 7: Net-(SW20-Pad1) -> Net-(SW60-Pad1)
- U9 pad 9: Net-(SW34-Pad1) -> Net-(U9-Pad9)
Routing:
- net Net-(SW61-Pad1): track 0.00 -> 135.0 mm
- net Net-(SW60-Pad1): track 0.00 -> 119.5 mm
- net Net-(SW50-Pad1): track 0.00 -> 118.7 mm
- net Net-(SW49-Pad1): track 0.00 -> 108.8 mm
- net Net-(SW59-Pad1): track 0.00 -> 108.5 mm
- net Net-(SW58-Pad1): track 0.00 -> 106.3 mm
- net Net-(SW36-Pad1): track 0.00 -> 105.5 mm
- net Net-(SW48-Pad1): track 0.00 -> 103.1 mm
- net Net-(SW57-Pad1): track 0.00 -> 102.7 mm
- net Net-(SW35-Pad1): track 0.00 -> 95.9 mm
- net Net-(SW47-Pad1): track 0.00 -> 93.8 mm
- net Net-(SW46-Pad1): track 0.00 -> 91.2 mm
- net Net-(SW34-Pad1): track 0.00 -> 89.9 mm
- net Net-(SW45-Pad1): track 0.00 -> 88.6 mm
- net Net-(SW44-Pad1): track 0.00 -> 87.8 mm
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- added copper zone on B.Cu, net (none)

Commit message: Updated symbols for 74HC365; routed all buffer to switch connections
Connections:
- U12 pad 11: Net-(SW9-Pad1) -> Net-(SW23-Pad1)
- U12 pad 13: Net-(SW23-Pad1) -> Net-(SW37-Pad1)
- U12 pad 3: Net-(SW37-Pad1) -> Net-(SW51-Pad1)
- U12 pad 5: Net-(SW51-Pad1) -> Net-(SW9-Pad1)
- U13 pad 11: Net-(SW10-Pad1) -> Net-(SW24-Pad1)
- U13 pad 13: Net-(SW24-Pad1) -> Net-(SW38-Pad1)
- U13 pad 3: Net-(SW38-Pad1) -> Net-(SW52-Pad1)
- U13 pad 5: Net-(SW52-Pad1) -> Net-(SW62-Pad1)
- U13 pad 7: Net-(SW62-Pad1) -> Net-(SW10-Pad1)
- U14 pad 11: Net-(SW11-Pad1) -> Net-(SW25-Pad1)
- U14 pad 13: Net-(SW25-Pad1) -> Net-(SW39-Pad1)
- U14 pad 3: Net-(SW39-Pad1) -> Net-(SW53-Pad1)
- U14 pad 5: Net-(SW53-Pad1) -> Net-(SW11-Pad1)
- U15 pad 11: Net-(SW12-Pad1) -> Net-(SW26-Pad1)
- U15 pad 13: Net-(SW26-Pad1) -> Net-(SW40-Pad1)
- U15 pad 3: Net-(SW40-Pad1) -> Net-(SW54-Pad1)
- U15 pad 5: Net-(SW54-Pad1) -> Net-(SW63-Pad1)
- U15 pad 7: Net-(SW63-Pad1) -> Net-(SW12-Pad1)
- U16 pad 11: Net-(SW13-Pad1) -> Net-(SW27-Pad1)
- U16 pad 13: Net-(SW27-Pad1) -> Net-(SW41-Pad1)
- U16 pad 3: Net-(SW41-Pad1) -> Net-(SW55-Pad1)
- U16 pad 5: Net-(SW55-Pad1) -> Net-(SW64-Pad1)
- U16 pad 7: Net-(SW64-Pad1) -> Net-(SW13-Pad1)
- U17 pad 11: Net-(SW14-Pad1) -> Net-(SW65-Pad1)
- U17 pad 13: Net-(SW28-Pad1) -> Net-(SW56-Pad1)
- U17 pad 5: Net-(SW56-Pad1) -> Net-(SW28-Pad1)
- U17 pad 7: Net-(SW65-Pad1) -> Net-(SW14-Pad1)
Routing:
- net ROW3: track 3.17 -> 267.5 mm
- net ROW4: track 11.7 -> 268.9 mm
- net ROW1: track 3.17 -> 236.5 mm
- net ROW0: track 3.17 -> 231.8 mm
- net ROW2: track 3.17 -> 224.6 mm
- net Net-(SW62-Pad1): track 4.80 -> 136.7 mm
- net Net-(SW63-Pad1): track 4.80 -> 123.5 mm
- net Net-(SW51-Pad1): track 10.0 -> 124.4 mm
- net Net-(SW64-Pad1): track 4.80 -> 117.4 mm
- net Net-(SW52-Pad1): track 10.1 -> 119.6 mm
- net Net-(SW55-Pad1): track 10.1 -> 113.9 mm
- net Net-(SW65-Pad1): track 4.80 -> 108.5 mm
- net Net-(SW53-Pad1): track 10.0 -> 112.8 mm
- net Net-(SW54-Pad1): track 10.1 -> 105.4 mm
- net Net-(SW37-Pad1): track 15.4 -> 103.6 mm
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
Commit message: Attempted routing plan for column select traces
Routing:
- net /COL8: track 0.00 -> 126.6 mm
- net /COL9: track 0.00 -> 109.2 mm
- net /COL10: track 0.00 -> 91.8 mm
- net /COL11: track 0.00 -> 74.4 mm
- net /COL12: track 0.00 -> 57.0 mm
- net /COL13: track 0.00 -> 39.6 mm
- net ROW0: track 231.8 -> 261.2 mm, vias 0 -> 1
- net /COL0: track 0.00 -> 18.7 mm
- net /COL1: track 0.00 -> 15.9 mm
- net /COL2: track 0.00 -> 13.1 mm
- net /COL3: track 0.00 -> 10.3 mm
- net /COL4: track 0.00 -> 7.53 mm
- net /COL5: track 0.00 -> 4.73 mm
- net /COL7: track 0.00 -> 4.47 mm
- net /COL6: track 0.00 -> 3.20 mm
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